File: OpenSampler/Baos_Board.brd (EAGLE design)
At the start: 57.2 x 26 mm, 34 parts, among them U1 FRAM, U2 DS3231ST&R

Commit message: Add files via upload
Parts:
- removed C1: 1 nF, rcl:C0805
- R7: value 500 -> 4.7k
Connections:
- net GND: no longer C1.2
- net V_LATCH: no longer C1.1
Routing:
- net V_LATCH: track 105.8 -> 104.1 mm
Changed lines of the file:
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@@
 <drawing>
 <settings>
-<setting alwaysvectorfont="yes"/>
+<setting alwaysvectorfont="no"/>
 <setting verticaltext="up"/>
 </settings>
@@
 </autorouter>
 <elements>
-<element name="C1" library="rcl" library_urn="urn:adsk.eagle:library:334" package="C0805" package3d_urn="urn:adsk.eagle:package:23617/2" value="1 nF" x="8.41" y="9.29" smashed="yes">
-<attribute name="NAME" x="7.14" y="10.56" size="1.27" layer="25"/>
-<attribute name="SPICEPREFIX" value="C" x="30" y="-25" size="1.778" layer="27" display="off"/>
-<attribute name="VALUE" x="7.14" y="6.75" size="1.27" layer="27"/>
-</element>
 <element name="C2" library="adafruit" package="C0805" value="100nF" x="41.29" y="10.71" smashed="yes" rot="MR90">
 <attribute name="NAME" x="42.306" y="9.821" size="1.27" layer="26" rot="MR90"/>
@@
 <attribute name="VALUE" x="36.245" y="8.9" size="1.27" layer="27" rot="R180"/>
 </element>
-<element name="R7" library="rcl" library_urn="urn:adsk.eagle:library:334" package="R0805" package3d_urn="urn:adsk.eagle:package:23553/2" value="500" x="35.175" y="20.05" smashed="yes">
+<element name="R7" library="rcl" library_urn="urn:adsk.eagle:library:334" package="R0805" package3d_urn="urn:adsk.eagle:package:23553/2" value="4.7k" x="35.175" y="20.05" smashed="yes">
 <attribute name="NAME" x="34.54" y="21.32" size="1.27" layer="25"/>
 <attribute name="SPICEPREFIX" value="R" x="51.685" y="-14.24" size="1.778" layer="27" display="off"/>
@@
 <contactref element="FET_N1" pad="2"/>
 <contactref element="FET_N2" pad="2"/>
-<contactref element="C1" pad="2"/>
 <contactref element="LED1" pad="C"/>
 <contactref element="FET_N4" pad="2"/>
@@
 <via x="16" y="7" extent="1-16" drill="0.508"/>
 <via x="30" y="13" extent="1-16" drill="0.508"/>
+<wire x1="45" y1="21" x2="47.672" y2="18.47" width="0" layer="19" extent="16-16"/>
+<wire x1="47.855" y1="13.4594" x2="47.672" y2="18.47" width="0" layer="19" extent="16-16"/>
+<wire x1="49" y1="11" x2="47.855" y2="13.4594" width="0" layer="19" extent="16-16"/>
+<wire x1="40" y1="18" x2="45" y2="21" width="0" layer="19" extent="1-1"/>
+<wire x1="38" y1="13" x2="40" y2="18" width="0" layer="19" extent="1-1"/>
+<wire x1="41.29" y1="11.56" x2="38" y2="13" width="0" layer="19" extent="16-16"/>
+<wire x1="41" y1="8" x2="41.29" y2="11.56" width="0" layer="19" extent="16-16"/>
+<wire x1="34.58" y1="10.1" x2="38" y2="13" width="0" layer="19" extent="1-1"/>
+<wire x1="32.8" y1="9.4" x2="34.58" y2="10.1" width="0" layer="19" extent="1-1"/>
+<wire x1="30.3163" y1="9.825" x2="32.8" y2="9.4" width="0" layer="19" extent="16-16"/>
+<wire x1="30.3163" y1="11.095" x2="30.3163" y2="9.825" width="0" layer="19" extent="16-16"/>
+<wire x1="30.3163" y1="8.555" x2="30.3163" y2="9.825" width="0" layer="19" extent="16-16"/>
+<wire x1="30.3163" y1="7.285" x2="30.3163" y2="8.555" width="0" layer="19" extent="16-16"/>
+<wire x1="30.3163" y1="6.015" x2="30.3163" y2="7.285" width="0" layer="19" extent="16-16"/>
+<wire x1="30" y1="13" x2="30.3163" y2="11.095" width="0" layer="19" extent="16-16"/>
+<wire x1="32.5" y1="5" x2="30.3163" y2="6.015" width="0" layer="19" extent="16-16"/>
+<wire x1="27.58" y1="10.1" x2="30.3163" y2="9.825" width="0" layer="19" extent="1-16"/>
+<wire x1="37.78" y1="23.37" x2="40" y2="18" width="0" layer="19" extent="1-1"/>
+<wire x1="20.9437" y1="9.825" x2="27.58" y2="10.1" width="0" layer="19" extent="1-16"/>
+<wire x1="20.9437" y1="11.095" x2="20.9437" y2="9.825" width="0" layer="19" extent="16-16"/>
+<wire x1="20.9437" y1="8.555" x2="20.9437" y2="9.825" width="0" layer="19" extent="16-16"/>
+<wire x1="20.9437" y1="7.285" x2="20.9437" y2="8.555" width="0" layer="19" extent="16-16"/>
+<wire x1="18.29" y1="4.94" x2="20.9437" y2="7.285" width="0" layer="19" extent="16-16"/>
+<wire x1="16" y1="7" x2="18.29" y2="4.94" width="0" layer="19" extent="16-16"/>
+<wire x1="12.27" y1="7.99" x2="16" y2="7" width="0" layer="19" extent="1-1"/>
+<wire x1="9.36" y1="3.94" x2="12.27" y2="7.99" width="0" layer="19" extent="1-1"/>
+<wire x1="3" y1="6" x2="9.36" y2="3.94" width="0" layer="19" extent="1-1"/>
+<wire x1="-1.88" y1="11.93" x2="3" y2="6" width="0" layer="19" extent="1-1"/>
+<wire x1="13.86" y1="17.62" x2="20.9437" y2="11.095" width="0" layer="19" extent="16-16"/>
+<wire x1="22" y1="21" x2="13.86" y2="17.62" width="0" layer="19" extent="16-16"/>
 </signal>
 <signal name="N$2">
@@
 <contactref element="D2" pad="A"/>
 <contactref element="R12" pad="2"/>
-<contactref element="C1" pad="1"/>
 <contactref element="FET_N4" pad="3"/>
 <contactref element="TEST3" pad="1"/>
@@
 <wire x1="14.47" y1="12" x2="12.48" y2="13.99" width="0.2032" layer="1"/>
 <wire x1="12.48" y1="13.99" x2="10.49" y2="13.99" width="0.2032" layer="1"/>
-<wire x1="7.46" y1="10.96" x2="7.46" y2="9.29" width="0.2032" layer="1"/>
 <wire x1="10.49" y1="13.99" x2="7.46" y2="10.96" width="0.2032" layer="1"/>
 <wire x1="8.5" y1="18.8766625" x2="7.7" y2="19.6766625" width="0.2032" layer="16"/>

Commit message: Add files via upload
Parts:
- removed TEST2, TEST3, TEST5: (no value), pinhead:1X01
- removed U1: FRAM, power8:FPT-8P-M02
- added FRAM: FRAM, power8:FPT-8P-M02
- added JP3: (no value), adafruit:1X03
- R7: value 4.7k -> 500
- moved TEST6 2.12 mm to (-1.00, 10.0)
- moved LED1 1.12 mm to (45.2, 18.0), flipped to the top
- moved JP2 0.56 mm to (42.0, 3.00), turned to 0 degrees
- moved JP1 0.41 mm to (42.0, 23.3)
- renumbered U2 to RTC
Connections:
- net +12V: now also JP1.2; no longer JP1.1
- net +3V3: now also FRAM.8, JP1.4; no longer U1.8
- net GND: now also FRAM.4, JP1.1; no longer JP1.2, U1.4
- net LOAD_LV: now also JP3.3; no longer TEST5.1
- net RTC_ALM: now also JP3.1; no longer TEST2.1
- net SCL: now also FRAM.6; no longer U1.6
- net SDA: now also FRAM.5; no longer U1.5
- net V_LATCH: now also JP3.2; no longer TEST3.1
Routing:
- net SDA: track 29.0 -> 15.9 mm
- net SHDN: track 39.0 -> 46.2 mm
- net V_LATCH: track 104.1 -> 97.7 mm
- net ALM_READ: track 34.7 -> 39.9 mm, vias 3 -> 4
- net N$9: track 22.1 -> 25.7 mm, vias 1 -> 2
- net +3V3: track 48.8 -> 52.0 mm
- net +12V: track 41.9 -> 44.9 mm
- net LOAD_LV: track 27.7 -> 26.7 mm, vias 1 -> 0
- net REGULATOR: track 12.0 -> 12.7 mm
Other:
- board size 57.2 x 26 mm -> 57 x 26.1 mm
- board text added: "GND"
- board text added: "Load_LV"
- board text added: "RTC_ALM"
- board text added: "V_Latch"

Commit message: Add files via upload
Parts:
- R7: value 500 -> 4.7k
Changed lines of the file:
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@@
 <attribute name="VALUE" x="36.245" y="8.9" size="1.27" layer="27" rot="R180"/>
 </element>
-<element name="R7" library="rcl" library_urn="urn:adsk.eagle:library:334" package="R0805" package3d_urn="urn:adsk.eagle:package:23553/2" value="500" x="35.175" y="20.05" smashed="yes">
+<element name="R7" library="rcl" library_urn="urn:adsk.eagle:library:334" package="R0805" package3d_urn="urn:adsk.eagle:package:23553/2" value="4.7k" x="35.175" y="20.05" smashed="yes">
 <attribute name="NAME" x="32.64" y="21.22" size="1.27" layer="25"/>
 <attribute name="SPICEPREFIX" value="R" x="51.685" y="-14.24" size="1.778" layer="27" display="off"/>
