File: OpenSampler/Baos_Board.sch (EAGLE design)
At the start: 34 parts, among them U1 FRAM, U2 DS3231ST&R

Commit message: Add files via upload
Parts:
- removed C1: 1 nF, rcl:C-USC0805
- R7: value 500 -> 4.7k
Connections:
- net GND: no longer C1.2
- net V_LATCH: no longer C1.1
Changed lines of the file:
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@@
 <part name="FET_P2" library="transistor-small-signal" library_urn="urn:adsk.eagle:library:401" deviceset="BSS84" device="" package3d_urn="urn:adsk.eagle:package:28738/2"/>
 <part name="R6" library="rcl" library_urn="urn:adsk.eagle:library:334" deviceset="R-US_" device="R0805" package3d_urn="urn:adsk.eagle:package:23553/2" value="500"/>
-<part name="R7" library="rcl" library_urn="urn:adsk.eagle:library:334" deviceset="R-US_" device="R0805" package3d_urn="urn:adsk.eagle:package:23553/2" value="500"/>
+<part name="R7" library="rcl" library_urn="urn:adsk.eagle:library:334" deviceset="R-US_" device="R0805" package3d_urn="urn:adsk.eagle:package:23553/2" value="4.7k"/>
 <part name="GND3" library="supply1" library_urn="urn:adsk.eagle:library:371" deviceset="GND" device=""/>
 <part name="D1" library="adafruit" deviceset="DIODE" device="SOD-123"/>
-<part name="C1" library="rcl" library_urn="urn:adsk.eagle:library:334" deviceset="C-US" device="C0805" package3d_urn="urn:adsk.eagle:package:23617/2" value="1 nF"/>
-<part name="GND5" library="supply1" library_urn="urn:adsk.eagle:library:371" deviceset="GND" device=""/>
 <part name="FET_P4" library="transistor-small-signal" library_urn="urn:adsk.eagle:library:401" deviceset="BSS84" device="" package3d_urn="urn:adsk.eagle:package:28738/2"/>
 <part name="D2" library="adafruit" deviceset="DIODE" device="SOD-123"/>
@@
 <attribute name="VALUE" x="-35.56" y="8.89" size="1.27" layer="96"/>
 </instance>
-<instance part="C1" gate="G$1" x="63.5" y="5.08" smashed="yes">
-<attribute name="NAME" x="64.516" y="5.715" size="1.778" layer="95"/>
-<attribute name="VALUE" x="64.516" y="0.889" size="1.778" layer="96"/>
-</instance>
-<instance part="GND5" gate="1" x="63.5" y="-5.08" smashed="yes">
-<attribute name="VALUE" x="60.96" y="-7.62" size="1.778" layer="96"/>
-</instance>
 <instance part="FET_P4" gate="G$1" x="81.28" y="50.8" smashed="yes">
 <attribute name="NAME" x="83.82" y="50.8" size="1.778" layer="95"/>
@@
 <pinref part="GND3" gate="1" pin="GND"/>
 <wire x1="50.8" y1="27.94" x2="50.8" y2="22.86" width="0.1524" layer="91"/>
-</segment>
-<segment>
-<pinref part="C1" gate="G$1" pin="2"/>
-<pinref part="GND5" gate="1" pin="GND"/>
-<wire x1="63.5" y1="0" x2="63.5" y2="-2.54" width="0.1524" layer="91"/>
 </segment>
 <segment>
@@
 <pinref part="R12" gate="G$1" pin="2"/>
 <junction x="63.5" y="53.34"/>
-<pinref part="C1" gate="G$1" pin="1"/>
-<wire x1="63.5" y1="12.7" x2="63.5" y2="7.62" width="0.1524" layer="91"/>
-<junction x="63.5" y="12.7"/>
 <wire x1="-22.86" y1="12.7" x2="-22.86" y2="2.54" width="0.1524" layer="91"/>
 <pinref part="FET_N4" gate="G$1" pin="D"/>

Commit message: Add files via upload
Other:
- note added: "James Yang, Bao Nguyen"
- note added: "James Yang, Bao Nguyen OPEnS Lab OSU"
- note removed: "mitchell nelke"
- note removed: "mitchell nelke OPEnS Lab OSU"
Changed lines of the file:
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@@
 <sheet>
 <plain>
-<text x="76.2" y="-22.86" size="2.54" layer="97">mitchell nelke</text>
-<text x="104.14" y="-22.86" size="2.54" layer="97">OPEnS Lab OSU</text>
+<text x="76.2" y="-22.86" size="2.54" layer="97">James Yang, Bao Nguyen</text>
+<text x="132.08" y="-22.86" size="2.54" layer="97">OPEnS Lab OSU</text>
 <text x="106.68" y="-43.18" size="2.54" layer="97">1</text>
 <text x="170.18" y="-43.18" size="2.54" layer="97">1</text>
@@
 <text x="187.96" y="-66.04" size="2.54" layer="97">2</text>
 <text x="248.92" y="-66.04" size="2.54" layer="97">1</text>
-<text x="157.48" y="-48.26" size="2.54" layer="97">mitchell nelke OPEnS Lab OSU</text>
+<text x="157.48" y="-48.26" size="2.54" layer="97">James Yang, Bao Nguyen OPEnS Lab OSU</text>
 </plain>
 <instances>

Commit message: Add files via upload
Parts:
- removed TEST2, TEST3, TEST5: (no value), pinhead:PINHD-1X1
- added JP3: (no value), adafruit:PINHD-1X3
- renumbered U1 to FRAM, U2 to RTC
Connections:
- net +12V: now also JP1.2; no longer JP1.1
- net +3V3: now also JP1.4
- net GND: now also JP1.1; no longer JP1.2
- net LOAD_LV: now also JP3.3; no longer TEST5.1
- net RTC_ALM: now also JP3.1; no longer TEST2.1
- net V_LATCH: now also JP3.2; no longer TEST3.1
Other:
- note added: "mitchell nelke"
- note added: "mitchell nelke OPEnS Lab OSU"
- note removed: "James Yang, Bao Nguyen"
- note removed: "James Yang, Bao Nguyen OPEnS Lab OSU"
- moved on the sheet: JP1

Commit message: Add files via upload
Other:
- note added: "James Yang, Bao Nguyen"
- note added: "James Yang, Bao Nguyen OPEnS Lab OSU"
- note removed: "mitchell nelke"
- note removed: "mitchell nelke OPEnS Lab OSU"
Changed lines of the file:
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@@
 <sheet>
 <plain>
-<text x="76.2" y="-22.86" size="2.54" layer="97">mitchell nelke</text>
-<text x="104.14" y="-22.86" size="2.54" layer="97">OPEnS Lab OSU</text>
+<text x="76.2" y="-22.86" size="2.54" layer="97">James Yang, Bao Nguyen</text>
+<text x="132.08" y="-22.86" size="2.54" layer="97">OPEnS Lab OSU</text>
 <text x="106.68" y="-43.18" size="2.54" layer="97">1</text>
 <text x="170.18" y="-43.18" size="2.54" layer="97">1</text>
@@
 <text x="187.96" y="-66.04" size="2.54" layer="97">2</text>
 <text x="248.92" y="-66.04" size="2.54" layer="97">1</text>
-<text x="157.48" y="-48.26" size="2.54" layer="97">mitchell nelke OPEnS Lab OSU</text>
+<text x="157.48" y="-48.26" size="2.54" layer="97">James Yang, Bao Nguyen OPEnS Lab OSU</text>
 </plain>
 <instances>
