File: 3v3_V2/p7.1_3v3.brd (EAGLE design)
At the start: 26 x 73.5 mm, 23 parts, among them Q1 MOSFET-SOT23F, Q2 SSM3J3228R, U1 SN74LVC1G175DBVR, U2 DS3231ST&R

Commit message: Add files via upload
Parts:
- removed U$3: (no value), adafruit:CR1220-SMD
- added U$1: (no value), adafruit:CR1220-THM
- C6: device adafruit:C0805 -> adafruit:C1206
- moved C6 0.99 mm to (5.02, 12.9)
Connections:
- net GND: now also U$1.+1, U$1.+2; no longer U$3.-
- net V_BACKUP: now also U$1.-; no longer U$3.+$1, U$3.+$2
Routing:
- net V_BACKUP: track 62.3 -> 42.3 mm, vias 0 -> 1
- net GND: track 13.6 -> 14.4 mm
Changed lines of the file:
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@@
 <setting verticaltext="up"/>
 </settings>
-<grid distance="0.5" unitdist="mm" unit="mm" style="lines" multiple="1" display="no" altdistance="5" altunitdist="mil" altunit="mil"/>
+<grid distance="0.5" unitdist="mm" unit="mm" style="lines" multiple="1" display="yes" altdistance="5" altunitdist="mil" altunit="mil"/>
 <layers>
 <layer number="1" name="Top" color="4" fill="1" visible="yes" active="yes"/>
@@
 <layer number="43" name="vRestrict" color="2" fill="10" visible="yes" active="yes"/>
 <layer number="44" name="Drills" color="7" fill="1" visible="no" active="yes"/>
-<layer number="45" name="Holes" color="7" fill="1" visible="no" active="yes"/>
+<layer number="45" name="Holes" color="7" fill="1" visible="yes" active="yes"/>
 <layer number="46" name="Milling" color="3" fill="1" visible="no" active="yes"/>
 <layer number="47" name="Measures" color="7" fill="1" visible="no" active="yes"/>
@@
 <wire x1="26" y1="70.5" x2="0" y2="70.5" width="0" layer="20"/>
 <wire x1="0" y1="70.5" x2="0" y2="-3" width="0" layer="20"/>
+<hole x="2.75" y="62.5" drill="2"/>
+<hole x="23.5" y="62.5" drill="2"/>
+<dimension x1="3.3" y1="54.85" x2="3.05" y2="54.85" x3="3.175" y3="48.65" textsize="1.778" layer="1"/>
+<dimension x1="3" y1="54.75" x2="3" y2="62.5" x3="-2" y3="58.625" textsize="1.778" layer="1"/>
+<dimension x1="2.75" y1="62.5" x2="5" y2="62.5" x3="3.875" y3="60.5" textsize="1.778" layer="1"/>
+<dimension x1="22.75" y1="54.75" x2="22.75" y2="61.75" x3="25" y3="58.25" textsize="1.778" layer="1"/>
+<dimension x1="2.75" y1="62.5" x2="23.5" y2="62.5" x3="13.125" y3="72.5" textsize="1.778" layer="1"/>
 </plain>
 <attributes>
@@
 <attribute name="VALUE" x="10.42" y="19.527" size="1.27" layer="28" rot="MR0"/>
 </element>
-<element name="C6" library="adafruit" package="C0805" value="100nF" x="5.78" y="13.53" smashed="yes" rot="MR0">
-<attribute name="NAME" x="6.669" y="14.546" size="1.27" layer="26" rot="MR0"/>
-<attribute name="VALUE" x="6.669" y="11.244" size="1.27" layer="28" rot="MR0"/>
+<element name="C6" library="adafruit" library_urn="urn:adsk.eagle:library:420" package="C1206" package3d_urn="urn:adsk.eagle:package:6240335/1" value="100nF" x="5.018" y="12.895" smashed="yes" rot="MR0">
+<attribute name="NAME" x="5.907" y="13.911" size="1.27" layer="26" rot="MR0"/>
+<attribute name="VALUE" x="5.907" y="10.609" size="1.27" layer="28" rot="MR0"/>
 </element>
 <element name="CP" library="jumper" library_urn="urn:adsk.eagle:library:252" package="SJ" package3d_urn="urn:adsk.eagle:package:15471/1" value="" x="21.717" y="5.08" smashed="yes" rot="MR0">
@@
 <element name="U$2" library="bluefruit_m0" package="BLUEFRUIT_MO" value="BLUEFRUIT_M0" x="24.476" y="1.992" smashed="yes" rot="R90">
 <attribute name="NAME" x="13.046" y="18.502" size="1.27" layer="25" rot="R90"/>
-</element>
-<element name="U$3" library="adafruit" library_urn="urn:adsk.eagle:library:420" package="CR1220-SMD" package3d_urn="urn:adsk.eagle:package:6240665/1" value="" x="12.979" y="63.369" smashed="yes" rot="MR0">
-<attribute name="NAME" x="16.535" y="68.971" size="1.6764" layer="26" font="vector" rot="MR0"/>
-<attribute name="VALUE" x="17.297" y="58.819" size="1.6764" layer="28" font="vector" rot="MR0"/>
 </element>
 <element name="U1" library="eDNA" package="DBV6" value="SN74LVC1G175DBVR" x="11.79" y="16.74" smashed="yes" rot="MR180">
@@
 <attribute name="PROD_ID" value="DIO-11284" x="8.12" y="-1.73" size="1.778" layer="27" rot="R180" display="off"/>
 <attribute name="VALUE" x="8.12" y="-0.968" size="0.6096" layer="27" font="vector" ratio="20" rot="R180" align="top-center"/>
+</element>
+<element name="U$1" library="adafruit" library_urn="urn:adsk.eagle:library:420" package="CR1220-THM" package3d_urn="urn:adsk.eagle:package:6240666/1" value="" x="12.5" y="64" smashed="yes">
+<attribute name="NAME" x="8.944" y="69.602" size="1.6764" layer="25" font="vector"/>
+<attribute name="VALUE" x="8.182" y="59.45" size="1.6764" layer="27" font="vector"/>
 </element>
 </elements>
@@
 <wire x1="6.1872" y1="16.663325" x2="6.1872" y2="17.336675" width="0.2032" layer="16"/>
 <wire x1="6.1872" y1="17.336675" x2="6.663325" y2="17.8128" width="0.2032" layer="16"/>
-<wire x1="6.63" y1="16.220525" x2="6.1872" y2="16.663325" width="0.2032" layer="16"/>
 <wire x1="8.8128" y1="17.8128" x2="9" y2="18" width="0.2032" layer="16"/>
 <wire x1="6.663325" y1="17.8128" x2="8.8128" y2="17.8128" width="0.2032" layer="16"/>
-<wire x1="6.63" y1="13.53" x2="6.63" y2="16.220525" width="0.2032" layer="16"/>
+<wire x1="6.418" y1="12.895" x2="6.418" y2="15.53428125" width="0.2032" layer="16"/>
+<wire x1="6.418" y1="15.53428125" x2="6.1872" y2="16.663325" width="0.2032" layer="16"/>
 <wire x1="10" y1="20" x2="11.078" y2="20" width="0.2032" layer="1"/>
 </signal>
@@
 <contactref element="U2" pad="6"/>
 <contactref element="U2" pad="5"/>
-<contactref element="U$3" pad="-"/>
 <polygon width="0.2032" layer="1">
 <vertex x="0" y="70.5"/>
@@
 <wire x1="8.03736875" y1="16.88789375" x2="7.336675" y2="16.1872" width="0.2032" layer="1"/>
 <wire x1="7.336675" y1="16.1872" x2="5.6872" y2="16.1872" width="0.2032" layer="1"/>
-<wire x1="4.5" y1="15" x2="4.93" y2="14.57" width="0.2032" layer="16"/>
-<wire x1="4.93" y1="14.57" x2="4.93" y2="13.53" width="0.2032" layer="16"/>
+<wire x1="4.5" y1="15" x2="4.6512375" y2="14.8487625" width="0.2032" layer="16"/>
+<wire x1="4.6512375" y1="14.8487625" x2="3.618" y2="12.895" width="0.2032" layer="16"/>
 <wire x1="10.922" y1="5.309" x2="10.995659375" y2="5.235340625" width="0.2032" layer="16"/>
 <wire x1="10.995659375" y1="5.235340625" x2="10.995659375" y2="3.504340625" width="0.2032" layer="16"/>
@@
 <via x="7" y="6" extent="1-16" drill="0.508"/>
 <contactref element="D2" pad="A"/>
+<contactref element="U$1" pad="+1"/>
+<contactref element="U$1" pad="+2"/>
 </signal>
 <signal name="GPIO_READ" class="3">
@@
 <contactref element="SD_PIN" pad="1"/>
 <contactref element="U$2" pad="3V"/>
-<wire x1="11.0254" y1="47.7756" x2="4.191" y2="54.61" width="0.2032" layer="1"/>
-<wire x1="4.191" y1="54.864" x2="4.191" y2="54.61" width="0.2032" layer="1"/>
+<wire x1="4.191" y1="54.61" x2="11.0254" y2="47.7756" width="0.2032" layer="1"/>
 <wire x1="22.571" y1="12" x2="22.571" y2="11.517" width="0.2032" layer="1"/>
 <wire x1="22.571" y1="11.517" x2="23.206" y2="10.882" width="0.2032" layer="1"/>
@@
 <wire x1="11.0254" y1="25.98675625" x2="22" y2="15.01215625" width="0.2032" layer="1"/>
 <wire x1="22" y1="15.01215625" x2="22" y2="12.571" width="0.2032" layer="1"/>
+<wire x1="4.191" y1="54.864" x2="4.191" y2="54.61" width="0.2032" layer="1"/>
 </signal>
 <signal name="CD">
@@
 <signal name="V_BACKUP">
 <contactref element="U2" pad="14"/>
-<contactref element="U$3" pad="+$1"/>
-<contactref element="U$3" pad="+$2"/>
 <wire x1="17.3163" y1="31.615" x2="17.9386" y2="32.2373" width="0.2032" layer="16"/>
 <wire x1="17.9386" y1="32.2373" x2="19.9361125" y2="32.2373" width="0.2032" layer="16"/>
 <wire x1="19.9361125" y1="32.2373" x2="21.06" y2="33.3611875" width="0.2032" layer="16"/>
 <wire x1="21.06" y1="33.3611875" x2="21.06" y2="49" width="0.2032" layer="16"/>
-<wire x1="21.179" y1="63.369" x2="21.06" y2="63.25" width="0.2032" layer="16"/>
-<wire x1="6.131" y1="53" x2="5.414" y2="53.717" width="0.2032" layer="16"/>
-<wire x1="4.779" y1="63.369" x2="5.414" y2="62.734" width="0.2032" layer="16"/>
-<wire x1="5.414" y1="62.734" x2="5.414" y2="53.717" width="0.2032" layer="16"/>
-<wire x1="17.06" y1="53" x2="21.06" y2="49" width="0.2032" layer="16"/>
-<wire x1="6.131" y1="53" x2="17.06" y2="53" width="0.2032" layer="16"/>
 <wire x1="21.06" y1="55.64129375" x2="20.7772" y2="55.35849375" width="0.2032" layer="16"/>
 <wire x1="20.7772" y1="55.35849375" x2="20.7772" y2="54.36950625" width="0.2032" layer="16"/>
 <wire x1="20.7772" y1="54.36950625" x2="21.06" y2="54.08670625" width="0.2032" layer="16"/>
 <wire x1="21.06" y1="54.08670625" x2="21.06" y2="49" width="0.2032" layer="16"/>
-<wire x1="21.06" y1="63.25" x2="21.06" y2="55.64129375" width="0.2032" layer="16"/>
+<contactref element="U$1" pad="-"/>
+<wire x1="21.06" y1="57.5" x2="21.06" y2="55.64129375" width="0.2032" layer="16"/>
+<wire x1="12.5" y1="64" x2="13.25" y2="63.25" width="0.2032" layer="1"/>
+<wire x1="13.25" y1="63.25" x2="13.25" y2="59.5" width="0.2032" layer="1"/>
+<via x="13.25" y="59.5" extent="1-16" drill="0.508"/>
+<wire x1="13.25" y1="59.5" x2="15.25" y2="57.5" width="0.2032" layer="16"/>
+<wire x1="15.25" y1="57.5" x2="21.06" y2="57.5" width="0.2032" layer="16"/>
 </signal>
 <signal name="N$6" class="3">
