File: 3v3_V2/p7.1_3v3.brd (EAGLE design)
At the start: 24.4 x 82.6 mm, 22 parts, among them U2 DS3231ST&R

Commit message: Add files via upload
Parts:
- removed U$4: NOT_GATE, eDNA:SOT753
- added Q2: SSM3J3228R, M0_Power:SOT-23-3
- added R5: 10k, adafruit:R1206
Connections:
- net 3V3_EN: now also Q2.D, R5.1; no longer U$4.4
- net EN_: now also Q2.G; no longer U$4.2
- net GND: now also R5.2; no longer U$4.3
- net VBATT: now also Q2.S; no longer U$4.5
Routing:
- net EN_: track 16.1 -> 25.6 mm
- net 3V3_EN: track 18.5 -> 23.4 mm, vias 1 -> 2
- net VBATT: track 50.5 -> 52.6 mm
- net SHDN_FEATHER: track 35.4 -> 36.1 mm
