File: 3v3_V2/p7.1_3v3.sch (EAGLE design)
At the start: 23 parts, among them Q1 MOSFET-SOT23F, Q2 SSM3J3228R, U1 SN74LVC1G175DBVR, U2 DS3231ST&R

Commit message: Add files via upload
Parts:
- removed U$3: (no value), adafruit:CR1220SMT
- added U$1: (no value), adafruit:CR1220THM
- C6: device adafruit:C-USC0805 -> adafruit:C-USC1206
Connections:
- net GND: now also U$1.+, U$1.+1; no longer U$3.-
- net V_BACKUP: now also U$1.-; no longer U$3.+, U$3.+1
Changed lines of the file:
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@@
 <part name="U2" library="power8" deviceset="DS3231ST&amp;R" device=""/>
 <part name="GND13" library="supply1" library_urn="urn:adsk.eagle:library:371" deviceset="GND" device=""/>
-<part name="C6" library="adafruit" deviceset="C-US" device="C0805" value="100nF"/>
+<part name="C6" library="adafruit" library_urn="urn:adsk.eagle:library:420" deviceset="C-US" device="C1206" package3d_urn="urn:adsk.eagle:package:6240335/1" value="100nF"/>
 <part name="GND14" library="supply1" library_urn="urn:adsk.eagle:library:371" deviceset="GND" device=""/>
-<part name="U$3" library="adafruit" library_urn="urn:adsk.eagle:library:420" deviceset="CR1220" device="SMT" package3d_urn="urn:adsk.eagle:package:6240665/1"/>
 <part name="GND9" library="SparkFun-PowerSymbols" library_urn="urn:adsk.eagle:library:530" deviceset="GND" device=""/>
 <part name="U1" library="eDNA" deviceset="SN74LVC1G175DBVR" device=""/>
@@
 <part name="C3" library="BOARD2.1FEATHER" deviceset="C-US" device="C1206" package3d_urn="urn:adsk.eagle:package:6240335/1" value="100nF"/>
 <part name="D2" library="SparkFun-DiscreteSemi" library_urn="urn:adsk.eagle:library:514" deviceset="DIODE-ZENER" device="-MM3Z3V3T1G" package3d_urn="urn:adsk.eagle:package:38441/1" value="3.3V"/>
+<part name="U$1" library="adafruit" library_urn="urn:adsk.eagle:library:420" deviceset="CR1220" device="THM" package3d_urn="urn:adsk.eagle:package:6240666/1"/>
 </parts>
 <sheets>
@@
 <attribute name="VALUE" x="-71.12" y="144.78" size="1.778" layer="96"/>
 </instance>
-<instance part="U$3" gate="G$1" x="73.66" y="170.18" smashed="yes" rot="MR0">
-<attribute name="NAME" x="74.93" y="173.355" size="1.778" layer="95" rot="MR0"/>
-<attribute name="VALUE" x="74.93" y="165.1" size="1.778" layer="96" rot="MR0"/>
-</instance>
 <instance part="GND9" gate="1" x="93.98" y="160.02" smashed="yes">
 <attribute name="VALUE" x="93.98" y="159.766" size="1.778" layer="96" align="top-center"/>
@@
 <attribute name="NAME" x="88.138" y="61.976" size="1.778" layer="95" font="vector" rot="R90"/>
 <attribute name="VALUE" x="92.202" y="61.976" size="1.778" layer="96" font="vector" rot="R90" align="top-left"/>
+</instance>
+<instance part="U$1" gate="G$1" x="71.12" y="170.18" smashed="yes">
+<attribute name="NAME" x="69.85" y="173.355" size="1.778" layer="95"/>
+<attribute name="VALUE" x="69.85" y="165.1" size="1.778" layer="96"/>
 </instance>
 </instances>
@@
 </segment>
 <segment>
-<pinref part="U$3" gate="G$1" pin="-"/>
-<wire x1="78.74" y1="170.18" x2="93.98" y2="170.18" width="0.1524" layer="91"/>
+<wire x1="76.2" y1="170.18" x2="93.98" y2="170.18" width="0.1524" layer="91"/>
 <pinref part="GND9" gate="1" pin="GND"/>
 <wire x1="93.98" y1="170.18" x2="93.98" y2="162.56" width="0.1524" layer="91"/>
+<pinref part="U$1" gate="G$1" pin="+"/>
+<wire x1="76.2" y1="172.72" x2="76.2" y2="170.18" width="0.1524" layer="91"/>
+<pinref part="U$1" gate="G$1" pin="+1"/>
+<wire x1="76.2" y1="167.64" x2="76.2" y2="170.18" width="0.1524" layer="91"/>
+<junction x="76.2" y="170.18"/>
 </segment>
 </net>
@@
 <pinref part="U2" gate="A" pin="VBAT"/>
 <wire x1="22.86" y1="170.18" x2="66.04" y2="170.18" width="0.1524" layer="91"/>
-<wire x1="66.04" y1="170.18" x2="66.04" y2="172.72" width="0.1524" layer="91"/>
-<pinref part="U$3" gate="G$1" pin="+"/>
-<wire x1="66.04" y1="172.72" x2="68.58" y2="172.72" width="0.1524" layer="91"/>
-<wire x1="66.04" y1="170.18" x2="66.04" y2="167.64" width="0.1524" layer="91"/>
-<junction x="66.04" y="170.18"/>
-<pinref part="U$3" gate="G$1" pin="+1"/>
-<wire x1="66.04" y1="167.64" x2="68.58" y2="167.64" width="0.1524" layer="91"/>
-</segment>
-</net>
+<pinref part="U$1" gate="G$1" pin="-"/>
+</segment>
+</net>
