File: 3v3_V2/p7.1_3v3.sch (EAGLE design)
At the start: 22 parts, among them U2 DS3231ST&R

Commit message: Add files via upload
Parts:
- removed U$4: NOT_GATE, eDNA:NOT_GATE
- added Q2: SSM3J3228R, M0_Power:SSM3J3228R
- added R5: 10k, adafruit:R-US_R1206
Connections:
- net 3V3_EN: now also Q2.D, R5.1; no longer U$4.OUT
- net EN_: now also Q2.G; no longer U$4.IN
- net GND: now also R5.2; no longer U$4.GND
- net VBATT: now also Q2.S; no longer U$4.VCC
Other:
- moved on the sheet: SW1, TESTGND
Changed lines of the file:
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@@
 <part name="C1" library="BOARD2.1FEATHER" deviceset="C-US" device="C1206" package3d_urn="urn:adsk.eagle:package:6240335/1" value="100nF"/>
 <part name="GND7" library="supply1" library_urn="urn:adsk.eagle:library:371" deviceset="GND" device=""/>
-<part name="GND8" library="supply1" library_urn="urn:adsk.eagle:library:371" deviceset="GND" device=""/>
-<part name="U$4" library="eDNA" deviceset="NOT_GATE" device=""/>
 <part name="TESTGND" library="adafruitmodified" deviceset="PINHD-1X1" device="" package3d_urn="urn:adsk.eagle:package:6240654/1"/>
 <part name="GND3" library="SparkFun-PowerSymbols" library_urn="urn:adsk.eagle:library:530" deviceset="GND" device=""/>
@@
 <part name="U$3" library="adafruit" library_urn="urn:adsk.eagle:library:420" deviceset="CR1220" device="SMT" package3d_urn="urn:adsk.eagle:package:6240665/1"/>
 <part name="GND9" library="SparkFun-PowerSymbols" library_urn="urn:adsk.eagle:library:530" deviceset="GND" device=""/>
+<part name="GND11" library="supply1" library_urn="urn:adsk.eagle:library:371" deviceset="GND" device=""/>
+<part name="Q2" library="M0_Power" deviceset="SSM3J3228R" device=""/>
+<part name="R5" library="adafruit" library_urn="urn:adsk.eagle:library:420" deviceset="R-US_" device="R1206" package3d_urn="urn:adsk.eagle:package:6240569/1" value="10k"/>
 </parts>
 <sheets>
@@
 <text x="-73.66" y="154.94" size="2.54" layer="97" font="vector" rot="R90">Decoupling</text>
 <text x="63.5" y="91.44" size="1.778" layer="91">3.3V into D-Flip-Flop instead of VBATT (4.2V)</text>
-<text x="-99.06" y="48.26" size="1.778" layer="91">Manually Wake Up (Testing purpose_)</text>
+<text x="-101.6" y="66.04" size="1.778" layer="91">Manually Wake Up (Testing purpose_)</text>
 <text x="-33.02" y="38.1" size="1.778" layer="91">Manually probing headers (testing purpose)</text>
 </plain>
@@
 <attribute name="VALUE" x="93.98" y="17.78" size="1.778" layer="96"/>
 </instance>
-<instance part="GND8" gate="1" x="40.64" y="106.68" smashed="yes">
-<attribute name="VALUE" x="38.1" y="104.14" size="1.778" layer="96"/>
-</instance>
-<instance part="U$4" gate="G$1" x="60.96" y="114.3" smashed="yes">
-<attribute name="VALUE" x="63.5" y="106.68" size="1.778" layer="96"/>
-<attribute name="NAME" x="63.5" y="121.92" size="1.778" layer="95"/>
-</instance>
-<instance part="TESTGND" gate="G$1" x="-45.72" y="20.32" smashed="yes">
-<attribute name="NAME" x="-52.07" y="23.495" size="1.778" layer="95"/>
-<attribute name="VALUE" x="-52.07" y="15.24" size="1.778" layer="96"/>
-</instance>
-<instance part="GND3" gate="1" x="-53.34" y="15.24" smashed="yes">
-<attribute name="VALUE" x="-53.34" y="14.986" size="1.778" layer="96" align="top-center"/>
-</instance>
-<instance part="SW1" gate="G$1" x="-68.58" y="40.64" smashed="yes">
-<attribute name="NAME" x="-71.12" y="44.196" size="1.27" layer="95"/>
-<attribute name="VALUE" x="-71.12" y="38.354" size="1.27" layer="96"/>
-</instance>
-<instance part="GND10" gate="1" x="-63.5" y="38.1" smashed="yes">
-<attribute name="VALUE" x="-63.5" y="37.846" size="1.778" layer="96" align="top-center"/>
+<instance part="TESTGND" gate="G$1" x="-48.26" y="38.1" smashed="yes">
+<attribute name="NAME" x="-54.61" y="41.275" size="1.778" layer="95"/>
+<attribute name="VALUE" x="-54.61" y="33.02" size="1.778" layer="96"/>
+</instance>
+<instance part="GND3" gate="1" x="-55.88" y="33.02" smashed="yes">
+<attribute name="VALUE" x="-55.88" y="32.766" size="1.778" layer="96" align="top-center"/>
+</instance>
+<instance part="SW1" gate="G$1" x="-71.12" y="58.42" smashed="yes">
+<attribute name="NAME" x="-73.66" y="61.976" size="1.27" layer="95"/>
+<attribute name="VALUE" x="-73.66" y="56.134" size="1.27" layer="96"/>
+</instance>
+<instance part="GND10" gate="1" x="-66.04" y="55.88" smashed="yes">
+<attribute name="VALUE" x="-66.04" y="55.626" size="1.778" layer="96" align="top-center"/>
 </instance>
 <instance part="U$3" gate="G$1" x="73.66" y="170.18" smashed="yes" rot="R180">
@@
 <instance part="GND9" gate="1" x="78.74" y="160.02" smashed="yes">
 <attribute name="VALUE" x="78.74" y="159.766" size="1.778" layer="96" align="top-center"/>
+</instance>
+<instance part="GND11" gate="1" x="68.58" y="106.68" smashed="yes">
+<attribute name="VALUE" x="66.04" y="104.14" size="1.778" layer="96"/>
+</instance>
+<instance part="Q2" gate="G$1" x="68.58" y="127" smashed="yes"/>
+<instance part="R5" gate="G$1" x="68.58" y="114.3" smashed="yes" rot="R270">
+<attribute name="NAME" x="70.0786" y="118.11" size="1.778" layer="95" rot="R270"/>
+<attribute name="VALUE" x="65.278" y="118.11" size="1.778" layer="96" rot="R270"/>
 </instance>
 </instances>
@@
 </segment>
 <segment>
-<label x="35.56" y="114.3" size="1.778" layer="95" rot="R180" xref="yes"/>
-<pinref part="U$4" gate="G$1" pin="VCC"/>
-<wire x1="38.1" y1="114.3" x2="55.88" y2="114.3" width="0.1524" layer="91"/>
+<pinref part="Q2" gate="G$1" pin="S"/>
+<wire x1="68.58" y1="132.08" x2="68.58" y2="134.62" width="0.1524" layer="91"/>
+<label x="68.58" y="134.62" size="1.778" layer="95" rot="R90" xref="yes"/>
 </segment>
 </net>
@@
 <segment>
 <pinref part="SW1" gate="G$1" pin="P$1"/>
-<wire x1="-73.66" y1="40.64" x2="-78.74" y2="40.64" width="0.1524" layer="91"/>
-<label x="-78.74" y="40.64" size="1.778" layer="95" rot="R180" xref="yes"/>
+<wire x1="-76.2" y1="58.42" x2="-81.28" y2="58.42" width="0.1524" layer="91"/>
+<label x="-81.28" y="58.42" size="1.778" layer="95" rot="R180" xref="yes"/>
 </segment>
 </net>
@@
 </segment>
 <segment>
-<pinref part="GND8" gate="1" pin="GND"/>
-<pinref part="U$4" gate="G$1" pin="GND"/>
-<wire x1="40.64" y1="109.22" x2="40.64" y2="111.76" width="0.1524" layer="91"/>
-<wire x1="40.64" y1="111.76" x2="55.88" y2="111.76" width="0.1524" layer="91"/>
-</segment>
-<segment>
 <pinref part="TESTGND" gate="G$1" pin="1"/>
-<wire x1="-48.26" y1="20.32" x2="-53.34" y2="20.32" width="0.1524" layer="91"/>
+<wire x1="-50.8" y1="38.1" x2="-55.88" y2="38.1" width="0.1524" layer="91"/>
 <pinref part="GND3" gate="1" pin="GND"/>
-<wire x1="-53.34" y1="20.32" x2="-53.34" y2="17.78" width="0.1524" layer="91"/>
+<wire x1="-55.88" y1="38.1" x2="-55.88" y2="35.56" width="0.1524" layer="91"/>
 </segment>
 <segment>
@@
 <wire x1="78.74" y1="170.18" x2="78.74" y2="162.56" width="0.1524" layer="91"/>
 <pinref part="U$3" gate="G$1" pin="-"/>
+</segment>
+<segment>
+<pinref part="R5" gate="G$1" pin="2"/>
+<pinref part="GND11" gate="1" pin="GND"/>
 </segment>
 </net>
@@
 </segment>
 <segment>
-<label x="43.18" y="116.84" size="1.778" layer="95" rot="R180" xref="yes"/>
-<pinref part="U$4" gate="G$1" pin="IN"/>
-<wire x1="43.18" y1="116.84" x2="55.88" y2="116.84" width="0.1524" layer="91"/>
+<label x="43.18" y="127" size="1.778" layer="95" rot="R180" xref="yes"/>
+<pinref part="Q2" gate="G$1" pin="G"/>
+<wire x1="55.88" y1="127" x2="58.42" y2="127" width="0.1524" layer="91"/>
+<wire x1="43.18" y1="127" x2="58.42" y2="127" width="0.1524" layer="91"/>
+<junction x="58.42" y="127"/>
 </segment>
 </net>
@@
 </segment>
 <segment>
-<label x="88.9" y="114.3" size="1.778" layer="95" xref="yes"/>
-<wire x1="81.28" y1="114.3" x2="88.9" y2="114.3" width="0.1524" layer="91"/>
-<pinref part="U$4" gate="G$1" pin="OUT"/>
-</segment>
-</net>
+<label x="86.36" y="119.38" size="1.778" layer="95" xref="yes"/>
+<pinref part="Q2" gate="G$1" pin="D"/>
+<pinref part="R5" gate="G$1" pin="1"/>
+<wire x1="68.58" y1="121.92" x2="68.58" y2="119.38" width="0.1524" layer="91"/>
+<junction x="68.58" y="119.38"/>
+<wire x1="68.58" y1="119.38" x2="86.36" y2="119.38" width="0.1524" layer="91"/>
+</segment>
+</net>
