File: 3v3_V3/p7.1_3v3.brd (EAGLE design)
At the start: 27.8 x 61.8 mm, 17 parts, among them Q1 SSM3J3228R, Q2 SSM3J3228R, U2 DS3231ST&R

Commit message: Add files via upload
Parts:
- moved Q2 0.36 mm to (25.7, 0.46)
Connections:
- removed net 3V: MS1.2
- new net 0RX: MS1.14, U$2.0RX
- new net 11: MS1.23, U$2.11
- new net 13: MS1.25, U$2.13
- new net 1TX: MS1.15, U$2.1TX
- new net 9: MS1.21, U$2.9
- new net A0: MS1.5, U$2.A0
- new net A1: MS1.6, U$2.A1
- new net A2: MS1.7, U$2.A2
- new net A3: MS1.8, U$2.A3
- new net ARF: MS1.3, U$2.ARF
- new net DFU: MS1.16, U$2.DFU
- new net EN: MS1.27, U$2.EN
- new net N$7: MS1.20
- new net N$8: MS1.19
- new net RESET: MS1.1, U$2.RST
- net 3VRAIL: now also EXT|RTC_INT.1, MS1.2
- net 5VRAIL: now also EXT|RTC_INT.2, MS1.26
- net RTC_INT: no longer EXT|RTC_INT.2
Routing:
- net 5VRAIL: track 0.00 -> 102.4 mm, vias 0 -> 3
- net OUTPUT3V3: track 0.00 -> 88.7 mm, vias 0 -> 2
- net 3VRAIL: track 0.00 -> 55.5 mm
- net N$2: track 0.00 -> 45.5 mm, vias 0 -> 2
- net DI: track 0.00 -> 39.6 mm, vias 0 -> 2
- net CLK: track 0.00 -> 38.8 mm, vias 0 -> 2
- net DO: track 0.00 -> 38.6 mm, vias 0 -> 1
- net 5VUSB: track 0.00 -> 36.4 mm
- net VBATT: track 0.00 -> 34.5 mm
- net CS: track 0.00 -> 33.1 mm, vias 0 -> 1
- net SDA: track 0.00 -> 32.9 mm, vias 0 -> 1
- net SCL: track 0.00 -> 31.3 mm, vias 0 -> 1
- net +3V3: track 0.00 -> 30.7 mm, vias 0 -> 1
- net RTC_INT: track 0.00 -> 17.6 mm
- net N$3: track 0.00 -> 12.6 mm
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- added copper zone on layer 1, net GND
- added copper zone on layer 16, net GND

Commit message: Add files via upload
Parts:
- 30K_: value 10k -> 30k
- renumbered C6 to 100NF, EXT|RTC_INT to 3V|5V, Q1 to PMOS_, Q2 to PMOS, R2 to 30K, R5 to 30K_, READ1 to 5VRAIL, READ2 to 3VRAIL, SW1 to BUTTON, U$1 to MICROSD, U$2 to FEATHER, U$3 to BATTERY, U2 to RTC

Commit message: Add files via upload
Parts:
- removed READ, SHDN: (no value), jumper:SJ
Connections:
- removed net N$1: 5VRAIL.1, FEATHER.6
- removed net N$3: 3VRAIL.1, FEATHER.5
- removed net N$7: MS1.20
- removed net N$8: MS1.19
- removed net RTC_READ: READ.1
- removed net RTC_READ_OUT: FEATHER.A4, MS1.9, READ.2
- removed net SHDN_FEATHER: SHDN.1
- removed net SHDN_FEATHER_OUT: FEATHER.A5, MS1.10, SHDN.2
- new net 3V: 3VRAIL.1, FEATHER.5, MS1.19
- new net 5V: 5VRAIL.1, FEATHER.6, MS1.20
Routing:
- net 3V: track 0.00 -> 14.3 mm
- net N$3: track 12.6 -> 0.00 mm
- net SHDN_FEATHER_OUT: track 5.28 -> 0.00 mm
- net RTC_READ_OUT: track 5.12 -> 0.00 mm
- net 5V: track 0.00 -> 4.61 mm
- net N$1: track 4.57 -> 0.00 mm
Changed lines of the file:
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@@
 <drawing>
 <settings>
-<setting alwaysvectorfont="yes"/>
+<setting alwaysvectorfont="no"/>
 <setting verticaltext="up"/>
 </settings>
@@
 <layer number="14" name="Route14" color="22" fill="1" visible="no" active="no"/>
 <layer number="15" name="Route15" color="23" fill="1" visible="no" active="no"/>
-<layer number="16" name="Bottom" color="1" fill="1" visible="no" active="yes"/>
+<layer number="16" name="Bottom" color="1" fill="1" visible="yes" active="yes"/>
 <layer number="17" name="Pads" color="2" fill="1" visible="yes" active="yes"/>
 <layer number="18" name="Vias" color="2" fill="1" visible="yes" active="yes"/>
@@
 <attribute name="VALUE" x="18.542" y="50.8" size="1.27" layer="28" rot="MR90"/>
 </element>
-<element name="READ" library="jumper" library_urn="urn:adsk.eagle:library:252" package="SJ" package3d_urn="urn:adsk.eagle:package:15471/1" value="" x="20.32" y="27.432" smashed="yes" rot="MR270">
-<attribute name="NAME" x="19.177" y="29.083" size="1.27" layer="26" ratio="10" rot="MR270"/>
-<attribute name="VALUE" x="20.32" y="27.0319" size="0.02" layer="28" rot="MR270"/>
-</element>
-<element name="SHDN" library="jumper" library_urn="urn:adsk.eagle:library:252" package="SJ" package3d_urn="urn:adsk.eagle:package:15471/1" value="" x="20.32" y="33.02" smashed="yes" rot="MR270">
-<attribute name="NAME" x="19.177" y="34.671" size="1.27" layer="26" ratio="10" rot="MR270"/>
-<attribute name="VALUE" x="20.32" y="32.6199" size="0.02" layer="28" rot="MR270"/>
-</element>
 <element name="BUTTON" library="adafruit" library_urn="urn:adsk.eagle:library:420" package="PUSHBUTTON_SMD_SJ" package3d_urn="urn:adsk.eagle:package:6240956/1" value="" x="12.7" y="34.29" smashed="yes" rot="MR0">
 <attribute name="NAME" x="13.081" y="36.703" size="0.8128" layer="26" ratio="18" rot="MR270"/>
@@
 <wire x1="6" y1="28" x2="5.21" y2="27.21" width="0.2032" layer="16"/>
 <wire x1="6" y1="30.59" x2="6" y2="28" width="0.2032" layer="16"/>
-</signal>
-<signal name="SHDN_FEATHER" class="3">
-<contactref element="SHDN" pad="1"/>
 </signal>
 <signal name="GND">
@@
 <wire x1="17.7652" y1="2.24" x2="18.65" y2="2.24" width="0.2032" layer="16"/>
 </signal>
-<signal name="RTC_READ" class="3">
-<contactref element="READ" pad="1"/>
-</signal>
 <signal name="DO">
 <contactref element="MICROSD" pad="7"/>
@@
 <wire x1="16" y1="41" x2="18" y2="43" width="0.2032" layer="16"/>
 <wire x1="18" y1="43" x2="18" y2="46" width="0.2032" layer="16"/>
-</signal>
-<signal name="N$1">
-<contactref element="FEATHER" pad="6"/>
-<contactref element="5VRAIL" pad="1"/>
-<wire x1="2.54" y1="38.1" x2="2.57655" y2="38.1" width="0.2032" layer="16"/>
-<wire x1="6.541" y1="39.323" x2="6.588" y2="39.37" width="0.2032" layer="16"/>
-<wire x1="2.57655" y1="38.1" x2="3.79955" y2="39.323" width="0.2032" layer="16"/>
-<wire x1="3.79955" y1="39.323" x2="6.541" y2="39.323" width="0.2032" layer="16"/>
-</signal>
-<signal name="N$3">
-<contactref element="FEATHER" pad="5"/>
-<contactref element="3VRAIL" pad="1"/>
-<wire x1="2.54" y1="51.689" x2="2.159" y2="52.07" width="0.2032" layer="16"/>
-<wire x1="2.54" y1="40.64" x2="2.54" y2="41.55815625" width="0.2032" layer="16"/>
-<wire x1="2.54" y1="47.41084375" x2="2.54" y2="51.689" width="0.2032" layer="16"/>
-<wire x1="2.54" y1="41.55815625" x2="1.27" y2="42.82815625" width="0.2032" layer="16"/>
-<wire x1="1.27" y1="46.14084375" x2="2.54" y2="47.41084375" width="0.2032" layer="16"/>
-<wire x1="1.27" y1="42.82815625" x2="1.27" y2="46.14084375" width="0.2032" layer="16"/>
 </signal>
 <signal name="5VUSB">
@@
 <wire x1="10.251103125" y1="41.251103125" x2="10.251103125" y2="39.637896875" width="0.2032" layer="16"/>
 </signal>
-<signal name="SHDN_FEATHER_OUT">
-<contactref element="SHDN" pad="2"/>
-<contactref element="FEATHER" pad="A5"/>
-<contactref element="MS1" pad="10"/>
-<wire x1="22.86" y1="30.48" x2="22.907" y2="30.433" width="0.2032" layer="1"/>
-<wire x1="22.907" y1="30.433" x2="24.847" y2="30.433" width="0.2032" layer="1"/>
-<wire x1="20.32" y1="32.258" x2="22.098" y2="30.48" width="0.2032" layer="16"/>
-<wire x1="22.098" y1="30.48" x2="22.86" y2="30.48" width="0.2032" layer="16"/>
-</signal>
-<signal name="RTC_READ_OUT">
-<contactref element="READ" pad="2"/>
-<contactref element="FEATHER" pad="A4"/>
-<contactref element="MS1" pad="9"/>
-<wire x1="22.86" y1="27.94" x2="24.8" y2="27.94" width="0.2032" layer="1"/>
-<wire x1="24.8" y1="27.94" x2="24.847" y2="27.893" width="0.2032" layer="1"/>
-<wire x1="20.32" y1="26.67" x2="21.67" y2="26.67" width="0.2032" layer="16"/>
-<wire x1="22.86" y1="27.86" x2="22.86" y2="27.94" width="0.2032" layer="16"/>
-<wire x1="21.67" y1="26.67" x2="22.86" y2="27.86" width="0.2032" layer="16"/>
-</signal>
 <signal name="VBAT" class="3">
 <contactref element="MS1" pad="28"/>
@@
 <wire x1="4.48" y1="20.32" x2="4.527" y2="20.273" width="0.2032" layer="16"/>
 </signal>
-<signal name="N$7">
-<contactref element="MS1" pad="20"/>
-</signal>
-<signal name="N$8">
-<contactref element="MS1" pad="19"/>
-</signal>
 <signal name="13">
 <contactref element="FEATHER" pad="13"/>
@@
 <wire x1="2.587" y1="30.433" x2="4.527" y2="30.433" width="0.2032" layer="16"/>
 </signal>
+<signal name="5V">
+<contactref element="FEATHER" pad="6"/>
+<contactref element="5VRAIL" pad="1"/>
+<contactref element="MS1" pad="20"/>
+<wire x1="2.54" y1="38.1" x2="4.48" y2="38.1" width="0.2032" layer="16"/>
+<wire x1="4.48" y1="38.1" x2="4.527" y2="38.053" width="0.2032" layer="16"/>
+<wire x1="4.527" y1="38.053" x2="5.844" y2="39.37" width="0.2032" layer="16"/>
+<wire x1="5.844" y1="39.37" x2="6.588" y2="39.37" width="0.2032" layer="16"/>
+</signal>
+<signal name="3V">
+<contactref element="FEATHER" pad="5"/>
+<contactref element="3VRAIL" pad="1"/>
+<contactref element="MS1" pad="19"/>
+<wire x1="2.54" y1="40.64" x2="2.587" y2="40.593" width="0.1524" layer="1"/>
+<wire x1="2.587" y1="40.593" x2="4.527" y2="40.593" width="0.1524" layer="1"/>
+<wire x1="2.54" y1="40.64" x2="2.54" y2="41.74315625" width="0.2032" layer="16"/>
+<wire x1="1.524" y1="46.14084375" x2="2" y2="46.61684375" width="0.2032" layer="16"/>
+<wire x1="2.54" y1="41.74315625" x2="1.524" y2="42.75915625" width="0.2032" layer="16"/>
+<wire x1="1.524" y1="42.75915625" x2="1.524" y2="46.14084375" width="0.2032" layer="16"/>
+<wire x1="2" y1="47.62876875" x2="2.37123125" y2="48" width="0.2032" layer="16"/>
+<wire x1="2.159" y1="52.07" x2="2.37123125" y2="51.85776875" width="0.2032" layer="16"/>
+<wire x1="2.37123125" y1="51.85776875" x2="2.37123125" y2="48" width="0.2032" layer="16"/>
+<wire x1="2" y1="46.61684375" x2="2" y2="47.62876875" width="0.2032" layer="16"/>
+</signal>
 </signals>
