File: 3v3_V3/p7.1_3v3 - Adafruit Battery.sch (EAGLE design)
At the start: 15 parts

Commit message: Final update for 3.3V prototype
Parts:
- removed 30K: 10k, adafruit:R-US_R1206
- removed 30K_: 30k, adafruit:R-US_R1206
- removed BATTERY: (no value), adafruit:CR1220SMT
- removed BUTTON: (no value), adafruit:SWITCH_PUSHBUTTONSOFTTOUCHSMD_SJ
- removed PMOS, PMOS_: SSM3J3228R, M0_Power:SSM3J3228R
- added B1: CR1220, microbuilder:BATTERYCR1220_SMT
- added C1: 100nF, adafruit:C-USC1206
- added CS: SD Select, SparkFun-Jumpers:JUMPER-SMT_2_NC_TRACE_SILK
- added INT: (no value), adafruit:PINHD-1X1CB
- added NPN: SOT23, transistor:BC849
- added PMOS1, PMOS2: SSM3J3228R, M0_Power:SSM3J3228R
- added R1, R2: 30k, adafruit:R-US_R1206
- added R3: 2M, adafruit:R-US_R1206
- added R4: 80k, adafruit:R-US_R1206
- added R5: 20k, adafruit:R-US_R1206
- added R6, R7: 10k, adafruit:R-US_R1206
- added U$1, U$2: PUSH_BUTTON, eDNA:PUSH_BUTTON
- 3V|5V: device pinhead:PINHD-1X2 -> SparkFun-Connectors:CONN_021X02_NO_SILK
- renumbered 100NF to C3, TESTGND to GND
Connections:
- removed net 3V: 3VRAIL.1, FEATHER.5, MS1.GPIO5
- removed net 5V: 5VRAIL.1, FEATHER.6, MS1.GPIO6
- removed net OUTPUT3V3: 30K_.1, 3VRAIL.2, PMOS.G
- removed net VBAT: MS1.VBAT
- new net A4: FEATHER.A4, MS1.GPIOA4
- new net A5: FEATHER.A5, MS1.GPIOA5
- new net N$1: 5VRAIL.1, FEATHER.6
- new net N$10: PMOS1.G, R4.2, R5.1
- new net N$11: CS.1, FEATHER.10, MS1.GPIO10
- new net N$3: 3VRAIL.1, FEATHER.5
- new net N$4: 5VRAIL.2, R1.1, R3.1
- new net N$5: 3VRAIL.2, PMOS2.G, R2.1
- new net N$6: NPN.B, R3.2
- new net N$7: MS1.GPIO6
- new net N$8: MS1.GPIO5
- new net N$9: NPN.C, R5.2
- net +3V3: now also PMOS2.S, R2.2, R6.1, R7.1; no longer MICROSD.VDD, PMOS.S
- net 3VRAIL: now also C1.1, MICROSD.VDD, PMOS2.D; no longer PMOS.D
- net 5VRAIL: now also PMOS1.D; no longer 30K.1, 5VRAIL.2, PMOS_.D, PMOS_.G
- net 5VUSB: now also PMOS1.S, R4.1; no longer PMOS_.S
- net CS: now also CS.2; no longer FEATHER.10, MS1.GPIO10
- net GND: now also B1.-, C1.2, NPN.E, R1.2, U$1.P$1, U$2.P$2; no longer 30K.2, 30K_.2, BATTERY.-, BUTTON.P$2
- net N$2: now also B1.+; no longer BATTERY.+, BATTERY.+1
- net RESET: now also U$1.P$2
- net RTC_INT: now also INT.1, U$2.P$1; no longer BUTTON.P$1
- net SCL: now also R7.2
- net SDA: now also R6.2
- net VBATT: now also MS1.VBAT
Other:
- moved on the sheet: 3VRAIL, 3V|5V, 5VRAIL
