File: Archive/Hypnos V3 - November 2019/Hypnos V3.sch (EAGLE design)
At the start: 39 parts, among them Q1 NMOS, Q2 NMOS

Commit message: Hypnos V3 hardware fix
Added diode to Hypnos V3 to minimize leaking current from uSD card to 3VRAIL.
Add pdf for schematic Hypnos V2 + Hypnos V3
Updated bill of material to Hypnos V3
Parts:
- removed 3VRAIL1: (no value), jumper:SJ
- removed D1: (no value), semicon-smd-ipc:D-SOD123
- added R10: 30k, Resistor_Capacitor:WSLP1206R0500FEA
Connections:
- removed net VDD: 3VRAIL1.1, C1.1, D1.C, MICROSD.VDD
- net 3VRAIL: now also C1.1, MICROSD.VDD, R10.1; no longer 3VRAIL1.2, D1.A
- net CS: now also R10.2
Changed lines of the file:
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@@
 <part name="GND11" library="supply1" library_urn="urn:adsk.eagle:library:371" deviceset="GND" device=""/>
 <part name="MS2" library="adafruit" deviceset="FEATHERWING" device="" package3d_urn="urn:adsk.eagle:package:6240959/1"/>
+<part name="R10" library="Resistor_Capacitor" library_urn="urn:adsk.eagle:library:11396451" deviceset="WSLP1206R0500FEA" device="" package3d_urn="urn:adsk.eagle:package:10872898/2" value="30k"/>
 <part name="RTC_INT" library="SparkFun-Jumpers" library_urn="urn:adsk.eagle:library:528" deviceset="JUMPER-SMT_2_NC_TRACE" device="_SILK" package3d_urn="urn:adsk.eagle:package:39281/1" value=""/>
 <part name="PMOS3" library="eDNA" deviceset="P-MOSFET" device="" package3d_urn="urn:adsk.eagle:package:13489247/1"/>
@@
 <part name="GND16" library="supply1" library_urn="urn:adsk.eagle:library:371" deviceset="GND" device=""/>
 <part name="GND17" library="supply1" library_urn="urn:adsk.eagle:library:371" deviceset="GND" device=""/>
-<part name="D1" library="semicon-smd-ipc" library_urn="urn:adsk.eagle:library:353" deviceset="D-" device="SOD123" package3d_urn="urn:adsk.eagle:package:26308/2"/>
-<part name="3VRAIL1" library="jumper" library_urn="urn:adsk.eagle:library:252" deviceset="SJ" device="" package3d_urn="urn:adsk.eagle:package:15471/1"/>
 </parts>
 <sheets>
@@
 </instance>
 <instance part="MS2" gate="G$1" x="637.54" y="-612.14" smashed="yes" rot="R270" grouprefs="MOSFET_CIRCUITRY"/>
+<instance part="R10" gate="G$1" x="698.5" y="-629.92" smashed="yes" rot="R270" grouprefs="MOSFET_CIRCUITRY">
+<attribute name="NAME" x="699.9986" y="-626.11" size="1.778" layer="95" rot="R270"/>
+<attribute name="VALUE" x="695.198" y="-626.11" size="1.778" layer="96" rot="R270"/>
+</instance>
 <instance part="RTC_INT" gate="G$1" x="685.8" y="-637.54" smashed="yes" grouprefs="MOSFET_CIRCUITRY">
 <attribute name="VALUE" x="688.34" y="-638.048" size="1.778" layer="96" font="vector" align="top-left"/>
@@
 <instance part="GND17" gate="1" x="769.62" y="-624.84" smashed="yes">
 <attribute name="VALUE" x="767.08" y="-627.38" size="1.778" layer="96"/>
-</instance>
-<instance part="D1" gate="G$1" x="843.28" y="-553.72" smashed="yes" rot="R270" grouprefs="SDCARD">
-<attribute name="NAME" x="845.058" y="-551.18" size="1.778" layer="95" rot="R270"/>
-<attribute name="VALUE" x="839.597" y="-551.18" size="1.778" layer="96" rot="R270"/>
-</instance>
-<instance part="3VRAIL1" gate="1" x="838.2" y="-556.26" smashed="yes" rot="R90" grouprefs="SDCARD">
-<attribute name="NAME" x="837.946" y="-551.688" size="1.778" layer="95" rot="R90"/>
-<attribute name="VALUE" x="842.01" y="-558.8" size="1.778" layer="96" rot="R90"/>
 </instance>
 </instances>
@@
 <segment>
 <pinref part="CS" gate="G$1" pin="2"/>
-<wire x1="688.34" y1="-642.62" x2="701.04" y2="-642.62" width="0.1524" layer="91" grouprefs="MOSFET_CIRCUITRY"/>
+<wire x1="688.34" y1="-642.62" x2="698.5" y2="-642.62" width="0.1524" layer="91" grouprefs="MOSFET_CIRCUITRY"/>
 <label x="701.04" y="-642.62" size="1.778" layer="95" xref="yes" grouprefs="MOSFET_CIRCUITRY"/>
+<pinref part="R10" gate="G$1" pin="2"/>
+<wire x1="698.5" y1="-642.62" x2="701.04" y2="-642.62" width="0.1524" layer="91" grouprefs="MOSFET_CIRCUITRY"/>
+<wire x1="698.5" y1="-635" x2="698.5" y2="-642.62" width="0.1524" layer="91" grouprefs="MOSFET_CIRCUITRY"/>
+<junction x="698.5" y="-642.62" grouprefs="MOSFET_CIRCUITRY"/>
 </segment>
 </net>
@@
 </segment>
 <segment>
+<wire x1="843.28" y1="-561.34" x2="843.28" y2="-556.26" width="0.1524" layer="91" grouprefs="SDCARD"/>
+<pinref part="MICROSD" gate="G$1" pin="VDD"/>
+<label x="843.28" y="-556.26" size="1.778" layer="95" rot="R180" xref="yes" grouprefs="SDCARD"/>
+<pinref part="C1" gate="G$1" pin="1"/>
+<wire x1="843.28" y1="-561.34" x2="858.52" y2="-561.34" width="0.1524" layer="91" grouprefs="SDCARD"/>
+<junction x="843.28" y="-561.34" grouprefs="SDCARD"/>
+</segment>
+<segment>
 <pinref part="R9" gate="G$1" pin="2"/>
 <wire x1="777.24" y1="-678.18" x2="782.32" y2="-678.18" width="0.1524" layer="91" grouprefs="MOSFET_CIRCUITRY"/>
@@
 </segment>
 <segment>
-<pinref part="3VRAIL1" gate="1" pin="2"/>
-<pinref part="D1" gate="G$1" pin="A"/>
-<wire x1="838.2" y1="-551.18" x2="843.28" y2="-551.18" width="0.1524" layer="91" grouprefs="SDCARD"/>
-<wire x1="843.28" y1="-551.18" x2="843.28" y2="-543.56" width="0.1524" layer="91" grouprefs="SDCARD"/>
-<junction x="843.28" y="-551.18" grouprefs="SDCARD"/>
-<label x="843.28" y="-543.56" size="1.778" layer="95" rot="R90" xref="yes" grouprefs="SDCARD"/>
+<pinref part="R10" gate="G$1" pin="1"/>
+<wire x1="698.5" y1="-624.84" x2="698.5" y2="-619.76" width="0.1524" layer="91" grouprefs="MOSFET_CIRCUITRY"/>
+<label x="698.5" y="-619.76" size="1.778" layer="95" rot="R90" xref="yes" grouprefs="MOSFET_CIRCUITRY"/>
 </segment>
 </net>
@@
 </segment>
 </net>
-<net name="VDD" class="0">
-<segment>
-<pinref part="C1" gate="G$1" pin="1"/>
-<pinref part="D1" gate="G$1" pin="C"/>
-<wire x1="843.28" y1="-556.26" x2="843.28" y2="-561.34" width="0.1524" layer="91" grouprefs="SDCARD"/>
-<pinref part="3VRAIL1" gate="1" pin="1"/>
-<wire x1="838.2" y1="-561.34" x2="843.28" y2="-561.34" width="0.1524" layer="91"/>
-<junction x="843.28" y="-561.34"/>
-<pinref part="MICROSD" gate="G$1" pin="VDD"/>
-<wire x1="843.28" y1="-561.34" x2="858.52" y2="-561.34" width="0.1524" layer="91"/>
-</segment>
-</net>
