File: Hypnos/Hypnos V2.1.sch (EAGLE design)
At the start: 32 parts

Commit message: Update 3V trace for Hypnos V3
Route missing trace for V3
Add bStop layer for V2
Clean up some note on schematic V2 and V3
Other:
- note removed: "Change from V1 to V2: RTC is powered with 3v3 instead of Vbat Add red LED if rail are switched on"
Changed lines of the file:
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@@
 <?xml version="1.0" encoding="utf-8"?>
 <!DOCTYPE eagle SYSTEM "eagle.dtd">
-<eagle version="9.5.2">
+<eagle version="9.5.0">
 <drawing>
 <settings>
@@
 <text x="713.74" y="-660.4" size="1.778" layer="91" grouprefs="MOSFET_CIRCUITRY">30k</text>
 <text x="721.36" y="-637.54" size="1.778" layer="91" grouprefs="MOSFET_CIRCUITRY">30k</text>
-<text x="769.62" y="-579.12" size="2.54" layer="91">Change from V1 to V2:
-RTC is powered with 3v3 instead of Vbat
-Add red LED if rail are switched on</text>
 <text x="756.92" y="-665.48" size="1.778" layer="97">Voltage drop: 1.8V
 Should drive at 0.5mA</text>
@@
 <segment>
 <pinref part="CS" gate="G$1" pin="2"/>
-<wire x1="688.34" y1="-645.16" x2="698.5" y2="-645.16" width="0.1524" layer="91" grouprefs="MOSFET_CIRCUITRY"/>
+<wire x1="688.34" y1="-645.16" x2="701.04" y2="-645.16" width="0.1524" layer="91" grouprefs="MOSFET_CIRCUITRY"/>
 <label x="701.04" y="-645.16" size="1.778" layer="95" xref="yes" grouprefs="MOSFET_CIRCUITRY"/>
-<wire x1="698.5" y1="-645.16" x2="701.04" y2="-645.16" width="0.1524" layer="91" grouprefs="MOSFET_CIRCUITRY"/>
-<wire x1="698.5" y1="-637.54" x2="698.5" y2="-645.16" width="0.1524" layer="91" grouprefs="MOSFET_CIRCUITRY"/>
-<junction x="698.5" y="-645.16" grouprefs="MOSFET_CIRCUITRY"/>
 </segment>
 </net>
