File: Hypnos 12V/Hypnos V3.1.brd (EAGLE design)
At the start: 25.6 x 52.4 mm, 39 parts, among them Q1 NMOS, Q2 NMOS

Commit message: Update 3V trace for Hypnos V3
Route missing trace for V3
Add bStop layer for V2
Clean up some note on schematic V2 and V3
Routing:
- net 3VRAIL: track 75.0 -> 92.4 mm, vias 1 -> 3
- net +3V3: track 58.5 -> 46.3 mm, vias 2 -> 3
- net GND: vias 36 -> 35
Other:
- board text added: "Hypnos V3.1"
- board text removed: "Hypnos V3"
Changed lines of the file:
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@@
 <?xml version="1.0" encoding="utf-8"?>
 <!DOCTYPE eagle SYSTEM "eagle.dtd">
-<eagle version="9.5.2">
+<eagle version="9.5.0">
 <drawing>
 <settings>
-<setting alwaysvectorfont="no"/>
+<setting alwaysvectorfont="yes"/>
 <setting verticaltext="up"/>
 </settings>
@@
 <text x="12.18" y="17.66" size="1.016" layer="22" rot="MR270">Optional
 I2C Pull Up</text>
-<text x="18" y="5" size="1.4224" layer="16" ratio="15" rot="MR0">Hypnos V3</text>
-<text x="18" y="3.5" size="1.016" layer="22" rot="MR0">OpenSlab</text>
+<text x="18.8" y="5" size="1.4224" layer="16" ratio="15" rot="MR0">Hypnos V3.1</text>
+<text x="18.8" y="3.5" size="1.016" layer="22" rot="MR0">OpenSlab</text>
 <text x="11.79" y="19.71" size="1.016" layer="22" ratio="10" rot="MR180">SDCS</text>
 <text x="15.76" y="31.45" size="0.8128" layer="22" rot="MR0">INT</text>
@@
 <text x="25" y="2" size="0.9" layer="21" ratio="10">G</text>
 <text x="18.5" y="4.5" size="0.8128" layer="21">80k</text>
-<text x="18" y="2" size="1.016" layer="22" rot="MR0">Bao Nguyen</text>
-<text x="18" y="5" size="1.4224" layer="30" ratio="20" rot="MR0">Hypnos V3</text>
+<text x="18.8" y="2" size="1.016" layer="22" rot="MR0">Bao Nguyen</text>
+<text x="18.8" y="5" size="1.4224" layer="30" ratio="20" rot="MR0">Hypnos V3.1</text>
 <text x="12.79" y="25.71" size="1.016" layer="22" ratio="10" rot="MR180">RTC</text>
 <wire x1="26.5" y1="50" x2="26.5" y2="49.5" width="0.0762" layer="20"/>
@@
 <vertex x="0.5" y="0"/>
 </polygon>
-<via x="10.5" y="8.11" extent="1-16" drill="0.508"/>
+<via x="10.3" y="9.11" extent="1-16" drill="0.508"/>
 <via x="15.64" y="22.46" extent="1-16" drill="0.4"/>
 <contactref element="C1" pad="2"/>
@@
 <via x="17.4" y="9.6" extent="1-16" drill="0.4"/>
 <via x="17.4" y="8.4" extent="1-16" drill="0.4"/>
-<via x="17.4" y="7.2" extent="1-16" drill="0.4"/>
 <via x="15.89" y="41.76" extent="1-16" drill="0.4"/>
 <contactref element="MICROSD" pad="CD2"/>
@@
 <wire x1="16" y1="10.58" x2="15.83" y2="10.75" width="0.254" layer="16"/>
 <wire x1="15.83" y1="17.019934375" x2="15.83" y2="10.75" width="0.254" layer="16"/>
-<wire x1="14.85" y1="6.54" x2="14.7952" y2="6.4852" width="0.2032" layer="1"/>
 <wire x1="16.372" y1="19.25" x2="15.83" y2="18.708" width="0.2032" layer="16"/>
 <wire x1="15.83" y1="18.708" x2="15.83" y2="17.019934375" width="0.2032" layer="16"/>
@@
 <contactref element="PMOS2" pad="S"/>
 <contactref element="R2" pad="2"/>
-<wire x1="7.71" y1="40.39013125" x2="7.71" y2="18.29" width="0.3048" layer="16"/>
-<wire x1="7.71" y1="18.29" x2="11.03" y2="14.97" width="0.3048" layer="16"/>
 <wire x1="7.605065625" y1="40.495065625" x2="8.185" y2="41.075" width="0.3048" layer="16"/>
 <via x="8.185" y="41.075" extent="1-16" drill="0.508"/>
@@
 <wire x1="5.32553125" y1="44.3546" x2="3.5146" y2="44.3546" width="0.3048" layer="16"/>
 <wire x1="6.0546" y1="43.62553125" x2="5.32553125" y2="44.3546" width="0.3048" layer="16"/>
-<wire x1="7.605065625" y1="40.495065625" x2="7.51" y2="40.59013125" width="0.3048" layer="16"/>
-<wire x1="6.0546" y1="42.04553125" x2="7.51" y2="40.59013125" width="0.3048" layer="16"/>
-<wire x1="7.605065625" y1="40.495065625" x2="7.71" y2="40.39013125" width="0.3048" layer="16"/>
+<wire x1="6.0546" y1="42.04553125" x2="7.605065625" y2="40.495065625" width="0.3048" layer="16"/>
 <contactref element="RTC" pad="2"/>
 <contactref element="C3" pad="1"/>
@@
 <wire x1="14.46" y1="27.31" x2="11.94" y2="29.83" width="0.2032" layer="1"/>
 <via x="14.9" y="27.31" extent="1-16" drill="0.508"/>
-<wire x1="14.9" y1="27.31" x2="14.528" y2="26.938" width="0.2032" layer="16"/>
 <contactref element="MS2" pad="2"/>
 <wire x1="2.27" y1="43.11" x2="3.5146" y2="44.3546" width="0.3048" layer="16"/>
@@
 <vertex x="9" y="40.8"/>
 </polygon>
-<wire x1="17.5" y1="37.945" x2="11.94" y2="29.88" width="0" layer="19" extent="1-1"/>
+<wire x1="7.8" y1="40.30013125" x2="7.8" y2="30.4" width="0.3048" layer="16"/>
+<wire x1="7.8" y1="30.4" x2="8.915" y2="29.285" width="0.3048" layer="16"/>
+<wire x1="7.605065625" y1="40.495065625" x2="7.8" y2="40.30013125" width="0.3048" layer="16"/>
+<wire x1="12.0418" y1="29.785" x2="11.5418" y2="29.285" width="0.3048" layer="16"/>
+<wire x1="11.5418" y1="29.285" x2="8.915" y2="29.285" width="0.3048" layer="16"/>
+<via x="12.0418" y="29.785" extent="1-16" drill="0.508"/>
+<wire x1="12.0418" y1="29.785" x2="12.035" y2="29.785" width="0.3048" layer="1"/>
+<wire x1="12.035" y1="29.785" x2="11.94" y2="29.88" width="0.3048" layer="1"/>
 </signal>
 <signal name="N$2">
@@
 <contactref element="R7" pad="1"/>
 <contactref element="R6" pad="1"/>
-<wire x1="14.475" y1="11.48" x2="14.505" y2="14.97" width="0" layer="19" extent="16-16"/>
-<wire x1="3.82" y1="5.33" x2="14.475" y2="11.48" width="0" layer="19" extent="16-16"/>
+<via x="12.4" y="8.8" extent="1-16" drill="0.508"/>
+<wire x1="3.82" y1="5.33" x2="4.7954" y2="6.3054" width="0.3048" layer="16"/>
+<wire x1="4.7954" y1="6.3054" x2="5.32553125" y2="6.3054" width="0.3048" layer="16"/>
+<wire x1="11.5464" y1="7.9464" x2="12.4" y2="8.8" width="0.3048" layer="16"/>
+<wire x1="11.5464" y1="7.9464" x2="6.96653125" y2="7.9464" width="0.3048" layer="16"/>
+<wire x1="5.32553125" y1="6.3054" x2="6.96653125" y2="7.9464" width="0.3048" layer="16"/>
+<wire x1="12.4" y1="8.8" x2="13.2" y2="9.6" width="0.3048" layer="1"/>
+<wire x1="13.2" y1="9.6" x2="13.2" y2="10.6" width="0.3048" layer="1"/>
+<via x="13.2" y="10.6" extent="1-16" drill="0.508"/>
+<wire x1="14.475" y1="11.48" x2="14.475" y2="11.25" width="0.3048" layer="16"/>
+<wire x1="14.475" y1="11.25" x2="13.825" y2="10.6" width="0.3048" layer="16"/>
+<wire x1="13.2" y1="10.6" x2="13.825" y2="10.6" width="0.3048" layer="16"/>
+<wire x1="14.475" y1="11.48" x2="14.505" y2="11.51" width="0.3048" layer="16"/>
+<wire x1="14.505" y1="11.51" x2="14.505" y2="14.97" width="0.3048" layer="16"/>
 </signal>
 <signal name="5VRAIL">
