File: Hypnos V2.2/Hypnos V2.2.sch (EAGLE design)
At the start: 32 parts

Commit message: Hypnos 2.2 and 3.2
+Change solder bridge to always connected pad
+Remove solder bridge for D1 diode
Parts:
- removed 3VRAIL, 3VRAIL1, 5VRAIL: (no value), jumper:SJ
- added 3V, 5V: JUMPER-SMT_2_NC_TRACE_SILK, SparkFun-Jumpers:JUMPER-SMT_2_NC_TRACE_SILK
Connections:
- removed net N$5: 3VRAIL.2, PMOS2.G, R2.1
- new net 5V: 3V.2, PMOS2.G, R2.1
- net 3VRAIL: no longer 3VRAIL1.2
- net N$1: now also 5V.1; no longer 5VRAIL.1
- net N$3: now also 3V.1; no longer 3VRAIL.1
- net N$4: now also 5V.2; no longer 5VRAIL.2
- net VDD: no longer 3VRAIL1.1
Changed lines of the file:
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@@
 <part name="GND9" library="SparkFun-PowerSymbols" library_urn="urn:adsk.eagle:library:530" deviceset="GND" device=""/>
 <part name="MICROSD" library="adafruit" library_urn="urn:adsk.eagle:library:420" deviceset="MICROSD" device="" package3d_urn="urn:adsk.eagle:package:6240723/1"/>
-<part name="5VRAIL" library="jumper" library_urn="urn:adsk.eagle:library:252" deviceset="SJ" device="" package3d_urn="urn:adsk.eagle:package:15471/1"/>
-<part name="3VRAIL" library="jumper" library_urn="urn:adsk.eagle:library:252" deviceset="SJ" device="" package3d_urn="urn:adsk.eagle:package:15471/1"/>
 <part name="R2" library="Resistor_Capacitor" library_urn="urn:adsk.eagle:library:11396451" deviceset="WSLP1206R0500FEA" device="" package3d_urn="urn:adsk.eagle:package:10872898/2" value="30k"/>
 <part name="GND8" library="supply1" library_urn="urn:adsk.eagle:library:371" deviceset="GND" device=""/>
@@
 <part name="GND12" library="SparkFun-PowerSymbols" library_urn="urn:adsk.eagle:library:530" deviceset="GND" device=""/>
 <part name="D1" library="semicon-smd-ipc" library_urn="urn:adsk.eagle:library:353" deviceset="D-" device="SOD123" package3d_urn="urn:adsk.eagle:package:26308/2"/>
-<part name="3VRAIL1" library="jumper" library_urn="urn:adsk.eagle:library:252" deviceset="SJ" device="" package3d_urn="urn:adsk.eagle:package:15471/1"/>
+<part name="5V" library="SparkFun-Jumpers" library_urn="urn:adsk.eagle:library:528" deviceset="JUMPER-SMT_2_NC_TRACE" device="_SILK" package3d_urn="urn:adsk.eagle:package:39281/1" value=""/>
+<part name="3V" library="SparkFun-Jumpers" library_urn="urn:adsk.eagle:library:528" deviceset="JUMPER-SMT_2_NC_TRACE" device="_SILK" package3d_urn="urn:adsk.eagle:package:39281/1" value=""/>
 </parts>
 <sheets>
@@
 </instance>
 <instance part="MICROSD" gate="G$1" x="876.3" y="-551.18" smashed="yes" grouprefs="SDCARD"/>
-<instance part="5VRAIL" gate="1" x="690.88" y="-650.24" smashed="yes" grouprefs="MOSFET_CIRCUITRY">
-<attribute name="NAME" x="695.452" y="-649.986" size="1.778" layer="95"/>
-<attribute name="VALUE" x="688.34" y="-654.05" size="1.778" layer="96"/>
-</instance>
-<instance part="3VRAIL" gate="1" x="683.26" y="-652.78" smashed="yes" grouprefs="MOSFET_CIRCUITRY">
-<attribute name="NAME" x="680.72" y="-652.78" size="1.778" layer="95"/>
-<attribute name="VALUE" x="680.72" y="-656.59" size="1.778" layer="96"/>
-</instance>
 <instance part="R2" gate="G$1" x="713.74" y="-652.78" smashed="yes" rot="R90" grouprefs="MOSFET_CIRCUITRY">
 <attribute name="NAME" x="712.2414" y="-656.59" size="1.778" layer="95" rot="R90"/>
@@
 <attribute name="VALUE" x="839.597" y="-553.72" size="1.778" layer="96" rot="R270"/>
 </instance>
-<instance part="3VRAIL1" gate="1" x="838.2" y="-556.26" smashed="yes" rot="R90">
-<attribute name="NAME" x="837.946" y="-551.688" size="1.778" layer="95" rot="R90"/>
-<attribute name="VALUE" x="842.01" y="-558.8" size="1.778" layer="96" rot="R90"/>
+<instance part="5V" gate="G$1" x="690.88" y="-650.24" smashed="yes">
+<attribute name="NAME" x="693.42" y="-650.24" size="1.778" layer="95" font="vector"/>
+<attribute name="VALUE" x="693.42" y="-650.748" size="1.778" layer="96" font="vector" align="top-left"/>
+</instance>
+<instance part="3V" gate="G$1" x="683.26" y="-652.78" smashed="yes">
+<attribute name="NAME" x="685.8" y="-652.78" size="1.778" layer="95" font="vector"/>
+<attribute name="VALUE" x="685.8" y="-653.288" size="1.778" layer="96" font="vector" align="top-left"/>
 </instance>
 </instances>
@@
 <segment>
 <wire x1="675.64" y1="-650.24" x2="685.8" y2="-650.24" width="0.1524" layer="91" grouprefs="MOSFET_CIRCUITRY"/>
-<pinref part="5VRAIL" gate="1" pin="1"/>
 <pinref part="MS2" gate="G$1" pin="GPIO6"/>
+<pinref part="5V" gate="G$1" pin="1"/>
 </segment>
 </net>
@@
 <segment>
 <wire x1="675.64" y1="-652.78" x2="678.18" y2="-652.78" width="0.1524" layer="91" grouprefs="MOSFET_CIRCUITRY"/>
-<pinref part="3VRAIL" gate="1" pin="1"/>
 <pinref part="MS2" gate="G$1" pin="GPIO5"/>
+<pinref part="3V" gate="G$1" pin="1"/>
 </segment>
 </net>
@@
 <segment>
 <pinref part="D1" gate="G$1" pin="A"/>
-<wire x1="843.28" y1="-553.72" x2="843.28" y2="-551.18" width="0.1524" layer="91" grouprefs="SDCARD"/>
 <label x="843.28" y="-548.64" size="1.778" layer="95" rot="R90" xref="yes" grouprefs="SDCARD"/>
-<wire x1="843.28" y1="-551.18" x2="843.28" y2="-548.64" width="0.1524" layer="91" grouprefs="SDCARD"/>
-<wire x1="838.2" y1="-551.18" x2="843.28" y2="-551.18" width="0.1524" layer="91" grouprefs="SDCARD"/>
-<junction x="843.28" y="-551.18" grouprefs="SDCARD"/>
-<pinref part="3VRAIL1" gate="1" pin="2"/>
+<wire x1="843.28" y1="-553.72" x2="843.28" y2="-548.64" width="0.1524" layer="91" grouprefs="SDCARD"/>
 </segment>
 <segment>
@@
 </segment>
 </net>
-<net name="N$5" class="0">
-<segment>
-<pinref part="3VRAIL" gate="1" pin="2"/>
+<net name="5V" class="0">
+<segment>
 <wire x1="688.34" y1="-652.78" x2="708.66" y2="-652.78" width="0.1524" layer="91" grouprefs="MOSFET_CIRCUITRY"/>
 <wire x1="708.66" y1="-652.78" x2="708.66" y2="-657.86" width="0.1524" layer="91" grouprefs="MOSFET_CIRCUITRY"/>
@@
 <pinref part="PMOS2" gate="G$1" pin="G"/>
 <wire x1="713.74" y1="-657.86" x2="721.36" y2="-657.86" width="0.1524" layer="91" grouprefs="MOSFET_CIRCUITRY"/>
+<pinref part="3V" gate="G$1" pin="2"/>
 </segment>
 </net>
 <net name="N$4" class="0">
 <segment>
-<pinref part="5VRAIL" gate="1" pin="2"/>
 <wire x1="695.96" y1="-650.24" x2="708.66" y2="-650.24" width="0.1524" layer="91" grouprefs="MOSFET_CIRCUITRY"/>
 <wire x1="708.66" y1="-650.24" x2="708.66" y2="-632.46" width="0.1524" layer="91" grouprefs="MOSFET_CIRCUITRY"/>
@@
 <pinref part="U$3" gate="G$1" pin="G"/>
 <wire x1="718.82" y1="-632.46" x2="734.06" y2="-632.46" width="0.1524" layer="91"/>
+<pinref part="5V" gate="G$1" pin="2"/>
 </segment>
 </net>
@@
 <wire x1="843.28" y1="-561.34" x2="843.28" y2="-558.8" width="0.1524" layer="91" grouprefs="SDCARD"/>
 <junction x="843.28" y="-561.34" grouprefs="SDCARD"/>
-<wire x1="838.2" y1="-561.34" x2="843.28" y2="-561.34" width="0.1524" layer="91" grouprefs="SDCARD"/>
-<pinref part="3VRAIL1" gate="1" pin="1"/>
-</segment>
-</net>
+</segment>
+</net>
