File: Hypnos V3.2/Hypnos V3.2.sch (EAGLE design)
At the start: 37 parts, among them Q1 NMOS, Q2 NMOS

Commit message: Add another uSD part
BOM has a new part link for uSD slot
Parts:
- removed 3VRAIL1: (no value), jumper:SJ
Connections:
- net 3VRAIL: no longer 3VRAIL1.2
- net VDD: no longer 3VRAIL1.1
Changed lines of the file:
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@@
 <part name="Q2" library="eDNA" deviceset="NMOS" device="" package3d_urn="urn:adsk.eagle:package:13526746/1"/>
 <part name="D1" library="semicon-smd-ipc" library_urn="urn:adsk.eagle:library:353" deviceset="D-" device="SOD123" package3d_urn="urn:adsk.eagle:package:26308/2"/>
-<part name="3VRAIL1" library="jumper" library_urn="urn:adsk.eagle:library:252" deviceset="SJ" device="" package3d_urn="urn:adsk.eagle:package:15471/1"/>
 <part name="3V" library="SparkFun-Jumpers" library_urn="urn:adsk.eagle:library:528" deviceset="JUMPER-SMT_2_NC_TRACE" device="_SILK" package3d_urn="urn:adsk.eagle:package:39281/1" value=""/>
 <part name="5V" library="SparkFun-Jumpers" library_urn="urn:adsk.eagle:library:528" deviceset="JUMPER-SMT_2_NC_TRACE" device="_SILK" package3d_urn="urn:adsk.eagle:package:39281/1" value=""/>
@@
 <attribute name="NAME" x="845.058" y="-551.18" size="1.778" layer="95" rot="R270"/>
 <attribute name="VALUE" x="839.597" y="-551.18" size="1.778" layer="96" rot="R270"/>
-</instance>
-<instance part="3VRAIL1" gate="1" x="838.2" y="-556.26" smashed="yes" rot="R90" grouprefs="SDCARD">
-<attribute name="NAME" x="837.946" y="-551.688" size="1.778" layer="95" rot="R90"/>
-<attribute name="VALUE" x="842.01" y="-558.8" size="1.778" layer="96" rot="R90"/>
 </instance>
 <instance part="3V" gate="G$1" x="683.26" y="-650.24" smashed="yes">
@@
 </segment>
 <segment>
-<pinref part="3VRAIL1" gate="1" pin="2"/>
 <pinref part="D1" gate="G$1" pin="A"/>
-<wire x1="838.2" y1="-551.18" x2="843.28" y2="-551.18" width="0.1524" layer="91" grouprefs="SDCARD"/>
 <wire x1="843.28" y1="-551.18" x2="843.28" y2="-543.56" width="0.1524" layer="91" grouprefs="SDCARD"/>
-<junction x="843.28" y="-551.18" grouprefs="SDCARD"/>
 <label x="843.28" y="-543.56" size="1.778" layer="95" rot="R90" xref="yes" grouprefs="SDCARD"/>
 </segment>
@@
 <pinref part="D1" gate="G$1" pin="C"/>
 <wire x1="843.28" y1="-556.26" x2="843.28" y2="-561.34" width="0.1524" layer="91" grouprefs="SDCARD"/>
-<pinref part="3VRAIL1" gate="1" pin="1"/>
-<wire x1="838.2" y1="-561.34" x2="843.28" y2="-561.34" width="0.1524" layer="91"/>
 <junction x="843.28" y="-561.34"/>
 <pinref part="MICROSD" gate="G$1" pin="VDD"/>
