File: Hypnos V3.2/Hypnos V3.2.brd (EAGLE design)
At the start: 25.6 x 52.4 mm, 37 parts, among them Q1 NMOS, Q2 NMOS

Commit message: Add another uSD part
BOM has a new part link for uSD slot
Parts:
- removed 3VRAIL1: (no value), jumper:SJ
Connections:
- net 3VRAIL: no longer 3VRAIL1.2
- net VDD: no longer 3VRAIL1.1
Routing:
- net VDD: track 22.4 -> 20.3 mm
- net 3VRAIL: track 92.4 -> 90.5 mm
Changed lines of the file:
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@@
 <drawing>
 <settings>
-<setting alwaysvectorfont="yes"/>
+<setting alwaysvectorfont="no"/>
 <setting verticaltext="up"/>
 </settings>
@@
 <attribute name="VALUE" x="5.7" y="6.385" size="1.27" layer="27" rot="R180"/>
 </element>
-<element name="3VRAIL1" library="jumper" library_urn="urn:adsk.eagle:library:252" package="SJ" package3d_urn="urn:adsk.eagle:package:15471/1" value="" x="3.83" y="1.685" smashed="yes" rot="R180">
-<attribute name="NAME" x="5.481" y="0.542" size="1.27" layer="25" ratio="10" rot="R180"/>
-<attribute name="VALUE" x="3.4299" y="1.685" size="0.02" layer="27" rot="R180"/>
-</element>
 <element name="3V" library="SparkFun-Jumpers" library_urn="urn:adsk.eagle:library:528" package="SMT-JUMPER_2_NC_TRACE_SILK" package3d_urn="urn:adsk.eagle:package:39281/1" value="" x="10.2" y="34.4" smashed="yes">
 <attribute name="NAME" x="12.2" y="34.943" size="0.8128" layer="25" font="vector" ratio="10" align="bottom-center"/>
@@
 <wire x1="18.8079" y1="36.9536625" x2="18.67" y2="36.8157625" width="0.4064" layer="1"/>
 <wire x1="18.67" y1="36.8157625" x2="18.67" y2="36.5964" width="0.4064" layer="1"/>
-<contactref element="3VRAIL1" pad="2"/>
 <contactref element="D1" pad="2"/>
 <wire x1="3.82" y1="4.295" x2="2.735" y2="3.21" width="0.3048" layer="1"/>
 <wire x1="2.735" y1="3.21" x2="2.095" y2="3.21" width="0.3048" layer="1"/>
-<wire x1="2.095" y1="3.21" x2="3.068" y2="2.237" width="0.3048" layer="1"/>
-<wire x1="3.068" y1="2.237" x2="3.068" y2="1.685" width="0.3048" layer="1"/>
 <contactref element="R7" pad="1"/>
 <contactref element="R6" pad="1"/>
@@
 <contactref element="C1" pad="1"/>
 <contactref element="D1" pad="1"/>
-<contactref element="3VRAIL1" pad="1"/>
 <contactref element="MICROSD" pad="4"/>
-<wire x1="4.592" y1="1.685" x2="4.592" y2="2.307" width="0.3048" layer="1"/>
-<wire x1="4.592" y1="2.307" x2="5.495" y2="3.21" width="0.3048" layer="1"/>
-<wire x1="6.70270625" y1="1.7344" x2="5.495" y2="2.94210625" width="0.3048" layer="1"/>
+<wire x1="6.50270625" y1="1.9344" x2="5.495" y2="2.94210625" width="0.3048" layer="1"/>
 <wire x1="5.495" y1="3.21" x2="5.495" y2="2.94210625" width="0.3048" layer="1"/>
-<wire x1="6.70270625" y1="1.7344" x2="9.7344" y2="1.7344" width="0.3048" layer="1"/>
+<wire x1="6.50270625" y1="1.9344" x2="9.9344" y2="1.9344" width="0.3048" layer="1"/>
 <wire x1="12.65" y1="4.65" x2="12.65" y2="5.74" width="0.3048" layer="1"/>
-<wire x1="9.7344" y1="1.7344" x2="12.4" y2="4.4" width="0.3048" layer="1"/>
+<wire x1="9.9344" y1="1.9344" x2="12.4" y2="4.4" width="0.3048" layer="1"/>
 <wire x1="12.4" y1="4.4" x2="12.65" y2="4.65" width="0.3048" layer="1"/>
 <wire x1="22.44" y1="5" x2="21.84" y2="4.4" width="0.3048" layer="1"/>
