File: Hypnos V3.2/Hypnos V3.2.brd (EAGLE design)
At the start: 25.6 x 52.4 mm, 38 parts, among them Q1 NMOS, Q2 NMOS

Commit message: HardwareX documentation revision
Parts:
- FEATHERWING: value FEATHERWING -> SENSOR_PINOUT
- MS2: value FEATHERWING -> FEATHER_PINOUT
- PMOS1, PMOS2: value SSM3J3228R -> DMP3099L-7
- PMOS3: value P-MOSFET -> DMP3056LDM-7
- Q1, Q2: value NMOS -> DMN65D8L-7
- renumbered MS1 to FEATHERWING
