File: Hypnos V3.5/HypnosV3.5.brd (EAGLE design)
At the start: 26.5 x 59 mm, 39 parts, among them J1 MEM2051-00-195-00-A_REVD1MEM2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, Q1 DMN65D8L-7, Q2 DMN65D8L-7

Commit message: Add files via upload
Parts:
- added B1: CR1220, microbuilder:CR1220
- moved C2 64.3 mm to (2.50, -54.0)
- moved D2 64.3 mm to (10.0, -54.5)
- moved J1 58.0 mm to (8.00, -37.5)
- moved BT1 0.50 mm to (45.0, 46.5)
Connections:
- net GND: now also B1.-
- net N$2: now also B1.+$1; no longer BT1.+
Routing:
- net GND: track 22.1 -> 39.2 mm
- net N$2: track 26.0 -> 27.5 mm

Commit message: Add files via upload
Parts:
- moved C2 64.4 mm to (36.0, 1.00)
- moved D2 64.4 mm to (43.5, 0.50)
- moved J1 58.4 mm to (40.5, 11.0)
Other:
- board text added: "Hypnos V3.5"
- board text removed: "Bryson Goto"
Changed lines of the file:
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@@
 <drawing>
 <settings>
-<setting alwaysvectorfont="no"/>
+<setting alwaysvectorfont="yes"/>
 <setting verticaltext="up"/>
 </settings>
@@
 <text x="19.41" y="31.15" size="0.8128" layer="21">3k</text>
 <text x="25" y="2" size="0.9" layer="21" ratio="10">G</text>
-<text x="18.8" y="2" size="1.016" layer="22" rot="MR0">Bryson Goto</text>
-<text x="19.3" y="5" size="1.4224" layer="30" ratio="20" rot="MR0">Hypnos V3.3</text>
+<text x="19.3" y="5" size="1.4224" layer="30" ratio="20" rot="MR0">Hypnos V3.5</text>
 <text x="12.79" y="25.71" size="1.016" layer="22" ratio="10" rot="MR180">RTC</text>
 <wire x1="26.5" y1="50" x2="26.5" y2="49.5" width="0.0762" layer="20"/>
@@
 <attribute name="VALUE" x="35.5" y="38" size="1.27" layer="27" align="top-left"/>
 </element>
-<element name="J1" library="MEM2051-00-195-00-A_REVD1" package="GCT_MEM2051-00-195-00-A_REVD1" value="MEM2051-00-195-00-A_REVD1MEM2051-00-195-00-A_GCT_MEM2051-00-195-00-A" x="8" y="-37.5" smashed="yes">
-<attribute name="DESCRIPTION" value=" 9 (8 + 1) Position Card Connector microSD Surface Mount, Right Angle Gold, 1.95mm profile, Normally open switch, Push push, Top mount " x="-8.5" y="-11.5" size="1.778" layer="27" display="off"/>
-<attribute name="DIGI-KEY_PART_NUMBER" value="2073-MEM2051-00-195-00-ATR-ND" x="-8.5" y="-11.5" size="1.778" layer="27" display="off"/>
-<attribute name="MF" value="Global Connector Technology" x="-8.5" y="-11.5" size="1.778" layer="27" display="off"/>
-<attribute name="MP" value="MEM2051-00-195-00-A" x="-8.5" y="-11.5" size="1.778" layer="27" display="off"/>
-<attribute name="NAME" x="1.015" y="-26.959" size="1.27" layer="25"/>
-<attribute name="PACKAGE" value="None" x="-8.5" y="-11.5" size="1.778" layer="27" display="off"/>
-<attribute name="PURCHASE-URL" value="https://pricing.snapeda.com/search/part/MEM2051-00-195-00-A/?ref=eda" x="-8.5" y="-11.5" size="1.778" layer="27" display="off"/>
-<attribute name="VALUE" x="1.015" y="-28.61" size="1.27" layer="27"/>
-</element>
-<element name="D2" library="semicon-smd-ipc" library_urn="urn:adsk.eagle:library:353" package="SOD123" package3d_urn="urn:adsk.eagle:package:26308/2" value="" x="10" y="-54.5" smashed="yes">
-<attribute name="NAME" x="8.095" y="-52.595" size="1.27" layer="25"/>
-<attribute name="POPULARITY" value="0" x="-13" y="-28.5" size="1.778" layer="27" display="off"/>
-<attribute name="VALUE" x="8.095" y="-57.675" size="1.27" layer="27"/>
-</element>
-<element name="C2" library="adafruit" library_urn="urn:adsk.eagle:library:420" package="C1206" package3d_urn="urn:adsk.eagle:package:6240335/1" value="100nF" x="2.5" y="-54" smashed="yes">
-<attribute name="NAME" x="1.23" y="-52.857" size="1.27" layer="25"/>
-<attribute name="VALUE" x="1.23" y="-56.413" size="1.27" layer="27"/>
+<element name="J1" library="MEM2051-00-195-00-A_REVD1" package="GCT_MEM2051-00-195-00-A_REVD1" value="MEM2051-00-195-00-A_REVD1MEM2051-00-195-00-A_GCT_MEM2051-00-195-00-A" x="40.5" y="11" smashed="yes">
+<attribute name="DESCRIPTION" value=" 9 (8 + 1) Position Card Connector microSD Surface Mount, Right Angle Gold, 1.95mm profile, Normally open switch, Push push, Top mount " x="24" y="37" size="1.778" layer="27" display="off"/>
+<attribute name="DIGI-KEY_PART_NUMBER" value="2073-MEM2051-00-195-00-ATR-ND" x="24" y="37" size="1.778" layer="27" display="off"/>
+<attribute name="MF" value="Global Connector Technology" x="24" y="37" size="1.778" layer="27" display="off"/>
+<attribute name="MP" value="MEM2051-00-195-00-A" x="24" y="37" size="1.778" layer="27" display="off"/>
+<attribute name="NAME" x="33.515" y="21.541" size="1.27" layer="25"/>
+<attribute name="PACKAGE" value="None" x="24" y="37" size="1.778" layer="27" display="off"/>
+<attribute name="PURCHASE-URL" value="https://pricing.snapeda.com/search/part/MEM2051-00-195-00-A/?ref=eda" x="24" y="37" size="1.778" layer="27" display="off"/>
+<attribute name="VALUE" x="33.515" y="19.89" size="1.27" layer="27"/>
+</element>
+<element name="D2" library="semicon-smd-ipc" library_urn="urn:adsk.eagle:library:353" package="SOD123" package3d_urn="urn:adsk.eagle:package:26308/2" value="" x="43.5" y="0.5" smashed="yes">
+<attribute name="NAME" x="41.595" y="2.405" size="1.27" layer="25"/>
+<attribute name="POPULARITY" value="0" x="20.5" y="26.5" size="1.778" layer="27" display="off"/>
+<attribute name="VALUE" x="41.595" y="-2.675" size="1.27" layer="27"/>
+</element>
+<element name="C2" library="adafruit" library_urn="urn:adsk.eagle:library:420" package="C1206" package3d_urn="urn:adsk.eagle:package:6240335/1" value="100nF" x="36" y="1" smashed="yes">
+<attribute name="NAME" x="34.73" y="2.143" size="1.27" layer="25"/>
+<attribute name="VALUE" x="34.73" y="-1.413" size="1.27" layer="27"/>
 </element>
 </elements>
@@
 <wire x1="25.24" y1="5" x2="23.697" y2="2.36" width="0" layer="19" extent="1-1"/>
 <wire x1="52.85" y1="46.5" x2="20.55" y2="2.34" width="0" layer="19" extent="1-1"/>
-<wire x1="4.44" y1="-30.075" x2="52.85" y2="46.5" width="0" layer="19" extent="1-1"/>
-<wire x1="4.44" y1="-41.36" x2="4.44" y2="-30.075" width="0" layer="19" extent="1-1"/>
-<wire x1="8.84" y1="-40.76" x2="4.44" y2="-41.36" width="0" layer="19" extent="1-1"/>
-<wire x1="3.9" y1="-54" x2="4.44" y2="-41.36" width="0" layer="19" extent="1-1"/>
+<wire x1="36.94" y1="18.425" x2="52.85" y2="46.5" width="0" layer="19" extent="1-1"/>
+<wire x1="36.94" y1="7.14" x2="36.94" y2="18.425" width="0" layer="19" extent="1-1"/>
+<wire x1="41.34" y1="7.74" x2="36.94" y2="7.14" width="0" layer="19" extent="1-1"/>
+<wire x1="37.4" y1="1" x2="36.94" y2="7.14" width="0" layer="19" extent="1-1"/>
 </signal>
 <signal name="DO">
@@
 <wire x1="2.27" y1="20.25" x2="4.81" y2="20.25" width="0.254" layer="1"/>
 <contactref element="J1" pad="P5"/>
-<wire x1="11.55" y1="6.14" x2="5.54" y2="-41.16" width="0" layer="19" extent="1-1"/>
+<wire x1="11.55" y1="6.14" x2="38.04" y2="7.34" width="0" layer="19" extent="1-1"/>
 </signal>
 <signal name="CS">
@@
 <wire x1="14.505" y1="11.51" x2="14.505" y2="14.97" width="0.3048" layer="16"/>
 <contactref element="D2" pad="2"/>
-<wire x1="2.095" y1="3.21" x2="11.7" y2="-54.5" width="0" layer="19" extent="1-1"/>
+<wire x1="2.095" y1="3.21" x2="45.2" y2="0.5" width="0" layer="19" extent="1-1"/>
 </signal>
 <signal name="5VRAIL">
@@
 <contactref element="C2" pad="1"/>
 <contactref element="D2" pad="1"/>
-<wire x1="8.3" y1="-54.5" x2="1.1" y2="-54" width="0" layer="19" extent="1-1"/>
-<wire x1="6.64" y1="-41.36" x2="8.3" y2="-54.5" width="0" layer="19" extent="1-1"/>
-<wire x1="5.495" y1="3.21" x2="6.64" y2="-41.36" width="0" layer="19" extent="1-1"/>
+<wire x1="41.8" y1="0.5" x2="34.6" y2="1" width="0" layer="19" extent="1-1"/>
+<wire x1="39.14" y1="7.14" x2="41.8" y2="0.5" width="0" layer="19" extent="1-1"/>
+<wire x1="5.495" y1="3.21" x2="39.14" y2="7.14" width="0" layer="19" extent="1-1"/>
 </signal>
 <signal name="10">

Commit message: Add files via upload
Parts:
- removed B1: CR1220, microbuilder:CR1220
- removed C2: 100nF, adafruit:C1206
- removed D2: (no value), semicon-smd-ipc:SOD123
- removed J1: MEM2051-00-195-00-A_REVD1MEM2051-00-195-00-A_GCT_MEM2051-00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, MEM2051-00-195-00-A_REVD1:GCT_MEM2051-00-195-00-A_REVD1
- moved BT1 31.6 mm to (13.4, 46.9), flipped to the bottom, turned to 90 degrees
- moved Q2 2.85 mm to (11.0, 50.0)
- moved 5V 1.31 mm to (8.71, 42.7)
Connections:
- net 3VRAIL: no longer D2.2
- net CLK: no longer J1.P5
- net GND: no longer B1.-, C2.2, J1.CD, J1.P2, J1.P6
- net N$2: now also BT1.+; no longer B1.+$1
- net VDD: no longer C2.1, D2.1, J1.P4
Routing:
- net GND: track 39.2 -> 258.6 mm, vias 35 -> 30
- net N$2: track 27.5 -> 21.7 mm
- net N$4: track 18.6 -> 23.9 mm, vias 0 -> 2
- net N$1: track 39.0 -> 43.8 mm, vias 3 -> 5
- net N$15: track 11.9 -> 14.3 mm
- net N$10: track 9.84 -> 9.18 mm
Other:
- board size 26.5 x 59 mm -> 26.5 x 59.5 mm
- board text added: "Woo, Goto"
- board text removed: "Hypnos V3.3"

Commit message: Add files via upload
Parts:
- moved Q2 2.85 mm to (13.8, 49.6)
- moved R2 1.50 mm to (17.5, 35.0)
- moved 5V 1.31 mm to (10.0, 42.7)
- moved BT1 1.14 mm to (13.3, 48.0)
Routing:
- net GND: track 258.6 -> 214.5 mm, vias 30 -> 14
- net N$2: track 21.7 -> 38.0 mm
- net N$1: track 43.8 -> 38.2 mm, vias 5 -> 3
- net N$4: track 23.9 -> 18.6 mm, vias 2 -> 0
- net +3V3: track 46.3 -> 51.0 mm
- net 3VRAIL: track 90.5 -> 93.4 mm
- net N$15: track 14.3 -> 11.9 mm
- net N$5: track 12.4 -> 13.2 mm
- net N$10: track 9.18 -> 9.84 mm
- net HIGHVOLTAGE: track 18.4 -> 19.0 mm
Other:
- board size 26.5 x 59.5 mm -> 26.5 x 60.5 mm
- board text added: "Goto, Woo"
- board text removed: "Woo, Goto"
